File: OpenCharger/OpenCharger.kicad_pcb (KiCad board)
At the start: 2 copper layers, 193 x 99.1 mm, 54 parts, among them J1 Conn_01x02, J2 Conn_01x03, J3 Conn_01x02, J4 RJ45_LED, Q1 IPT015N10N5, Q2 IPT015N10N5, Q3 IPT015N10N5, Q4 IPT015N10N5, Q5 BS870, Q5 IPT015N10N5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

Commit message: hi
Parts:
- moved J4 258.9 mm to (363.5, 212.2)
- moved U1 258.9 mm to (367.0, 226.9)
- moved D6 165.2 mm to (209.6, 175.3)
- moved C5 165.1 mm to (193.0, 179.1)
- moved Q5 26.2 mm to (167.6, 207.0), turned to 90 degrees
- moved Q6 26.2 mm to (167.6, 238.8), turned to 90 degrees
- moved Q7 18.5 mm to (200.7, 238.8), turned to 90 degrees
- moved Q9 18.0 mm to (200.7, 207.0), turned to 90 degrees
Routing:
- added copper zone on B.Cu, net Earth
