File: OpenCharger/OpenCharger.kicad_pcb (KiCad board)
At the start: 2 copper layers, 193 x 99.1 mm, 54 parts, among them J1 Conn_01x02, J2 Conn_01x03, J3 Conn_01x02, J4 RJ45_LED, Q1 IPT015N10N5, Q2 IPT015N10N5, Q3 IPT015N10N5, Q4 IPT015N10N5, Q5 BS870, Q5 IPT015N10N5, Q6 IPT015N10N5, Q7 IPT015N10N5, Q8 IPT015N10N5, Q9 IPT015N10N5, U1 ISO1050DUB, U2 STM8AF6223A, U3 LMH6609MF, U4 IRS25606S, U5 LMH6609MF, Y1 Resonator_Small

Commit message: updated
Parts:
- removed D2, D5, D6: 15V, Diode_SMD:D_0603_1608Metric
- removed the Q5 at (314.7, 186.2)
- removed R13: R_US, Resistor_SMD:R_0603_1608Metric
- removed the R14 at (280.9, 195.8)
- removed the R15 at (314.7, 197.8)
- removed R3: 20k, Resistor_SMD:R_0603_1608Metric
- removed the R7 at (300.7, 198.4)
- removed the R7 at (228.9, 216.2)
- removed R9: 200k, Resistor_SMD:R_0603_1608Metric
- removed U5: LMH6609MF, Package_TO_SOT_SMD:SOT-23-5
- added C15: 100uF, Capacitor_THT:CP_Radial_D16.0mm_P7.50mm, F.Cu at (218.1, 248.3)
- added C16: 100uF, Capacitor_THT:CP_Radial_D16.0mm_P7.50mm, F.Cu at (218.1, 179.7)
- added C17: C, Capacitor_SMD:C_0603_1608Metric, F.Cu at (255.0, 87.0)
- added C6: 100uF, Capacitor_THT:CP_Radial_D16.0mm_P7.50mm, F.Cu at (218.1, 214.0)
- added IC1: INA211CQDCKRQ1, SamacSys_Parts:SOT65P210X110-6N, F.Cu at (288.8, 244.6)
- added IC10: 1EDI60N12AFXUMA1, SamacSys_Parts:SOIC127P600X175-8N, F.Cu at (205.6, 83.8)
- added IC11: 1EDI60N12AFXUMA1, SamacSys_Parts:SOIC127P600X175-8N, F.Cu at (214.1, 83.8)
- added IC12: 1EDI60N12AFXUMA1, SamacSys_Parts:SOIC127P600X175-8N, F.Cu at (222.6, 96.9)
- added IC13: 1EDI60N12AFXUMA1, SamacSys_Parts:SOIC127P600X175-8N, F.Cu at (214.1, 90.4)
- added IC2: 1EDI60N12AFXUMA1, SamacSys_Parts:SOIC127P600X175-8N, F.Cu at (222.6, 83.8)
- added IC3: 1EDI60N12AFXUMA1, SamacSys_Parts:SOIC127P600X175-8N, F.Cu at (222.6, 90.4)
- added IC4: 1EDI60N12AFXUMA1, SamacSys_Parts:SOIC127P600X175-8N, F.Cu at (197.1, 96.9)
- added IC5: 1EDI60N12AFXUMA1, SamacSys_Parts:SOIC127P600X175-8N, F.Cu at (197.1, 90.4)
- added IC6: 1EDI60N12AFXUMA1, SamacSys_Parts:SOIC127P600X175-8N, F.Cu at (178.6, 111.3)
- added IC7: 1EDI60N12AFXUMA1, SamacSys_Parts:SOIC127P600X175-8N, F.Cu at (205.6, 96.9)
- added IC8: 1EDI60N12AFXUMA1, SamacSys_Parts:SOIC127P600X175-8N, F.Cu at (205.6, 90.4)
- added IC9: 1EDI60N12AFXUMA1, SamacSys_Parts:SOIC127P600X175-8N, F.Cu at (214.1, 96.9)
- added J5: Conn_01x02, Connector_PinHeader_2.54mm:PinHeader_1x02_P2.54mm_Vertical, F.Cu at (247.7, 135.3)
- added J6: Conn_01x01_Female, Connector:Banana_Jack_1Pin, F.Cu at (90.7, 220.3)
- added J7: Conn_02x05_Odd_Even, Connector_PinHeader_2.54mm:PinHeader_2x05_P2.54mm_Vertical, F.Cu at (116.3, 281.4)
- added Q10: IPT015N10N5, Package_TO_SOT_SMD:Infineon_PG-HSOF-8-1, B.Cu at (109.7, 234.8)
- added Q11: IPT015N10N5, Package_TO_SOT_SMD:Infineon_PG-HSOF-8-1, B.Cu at (109.7, 248.8)
- added Q12: IPT015N10N5, Package_TO_SOT_SMD:Infineon_PG-HSOF-8-1, B.Cu at (109.7, 262.8)
- added Q13: IPT015N10N5, Package_TO_SOT_SMD:Infineon_PG-HSOF-8-1, B.Cu at (95.8, 177.7)
- added Q14: IPT015N10N5, Package_TO_SOT_SMD:Infineon_PG-HSOF-8-1, B.Cu at (95.8, 191.6)
- added Q15: IPT015N10N5, Package_TO_SOT_SMD:Infineon_PG-HSOF-8-1, B.Cu at (95.8, 205.6)
- added Q16: IPT015N10N5, Package_TO_SOT_SMD:Infineon_PG-HSOF-8-1, B.Cu at (95.8, 248.8)
- added Q17: IPT015N10N5, Package_TO_SOT_SMD:Infineon_PG-HSOF-8-1, B.Cu at (95.8, 262.8)
- added Q18: IPT015N10N5, Package_TO_SOT_SMD:Infineon_PG-HSOF-8-1, B.Cu at (175.3, 190.5)
- added Q19: IPT015N10N5, Package_TO_SOT_SMD:Infineon_PG-HSOF-8-1, B.Cu at (175.3, 204.5)
- added Q20: IPT015N10N5, Package_TO_SOT_SMD:Infineon_PG-HSOF-8-1, B.Cu at (175.3, 236.2)
- added Q21: IPT015N10N5, Package_TO_SOT_SMD:Infineon_PG-HSOF-8-1, B.Cu at (175.3, 250.2)
- added Q22: IPT015N10N5, Package_TO_SOT_SMD:Infineon_PG-HSOF-8-1, B.Cu at (188.0, 236.2)
- added Q23: IPT015N10N5, Package_TO_SOT_SMD:Infineon_PG-HSOF-8-1, B.Cu at (188.0, 250.2)
- added Q24: IPT015N10N5, Package_TO_SOT_SMD:Infineon_PG-HSOF-8-1, B.Cu at (188.0, 190.5)
- added Q25: IPT015N10N5, Package_TO_SOT_SMD:Infineon_PG-HSOF-8-1, B.Cu at (188.0, 176.5)
- added Q26: IPT015N10N5, Package_TO_SOT_SMD:Infineon_PG-HSOF-8-1, B.Cu at (221.6, 171.4)
- added R10: 10k, Resistor_SMD:R_0603_1608Metric, F.Cu at (255.8, 84.3)
- added R14: R_US, Resistor_SMD:R_0603_1608Metric, F.Cu at (246.9, 86.4)
- added R14: R_US, Resistor_SMD:R_0603_1608Metric, F.Cu at (298.1, 82.6)
- added R15: R_US, Resistor_SMD:R_0603_1608Metric, F.Cu at (246.9, 88.9)
- added R15: R_US, Resistor_SMD:R_0603_1608Metric, F.Cu at (298.1, 80.1)
- added R7: .1m, Resistor_SMD:R_4020_10251Metric, F.Cu at (284.5, 82.3)
- added R7: R_Shunt_US, SamacSys_Parts:WSK1216L2000FEA, F.Cu at (286.0, 142.2)
- C1, C2: footprint Capacitor_SMD:C_1206_3216Metric -> Capacitor_SMD:C_0603_1608Metric
- C10, C5, C8: value C -> 100uF; footprint Capacitor_SMD:C_1206_3216Metric -> Capacitor_THT:CP_Radial_D16.0mm_P7.50mm
- C12, C13, C14, C3, C4, C9: value 56uF -> 100uF; footprint Capacitor_THT:CP_Radial_D40.0mm_P10.00mm_SnapIn -> Capacitor_THT:CP_Radial_D16.0mm_P7.50mm
- D1: value 15V -> 5V
- J1: value Conn_01x02 -> Conn_01x01_Female; footprint Connector:Banana_Jack_2Pin -> Connector:Banana_Jack_1Pin
- J2: footprint Connector:Banana_Jack_3Pin -> Connector_PinHeader_2.54mm:PinHeader_1x03_P2.54mm_Vertical
- R1: value 20k -> 1k
- R17, R18: value R_US -> 99k
- R2, R4: value 20k -> R_US
- R8: value 20k -> R_Small_US; footprint Resistor_SMD:R_0603_1608Metric -> Resistor_SMD:R_1206_3216Metric
- U4: value IRS25606S -> MCP6L01x-xLT; footprint Package_SO:SOIC-8_3.9x4.9mm_P1.27mm -> Package_TO_SOT_SMD:SOT-353_SC-70-5
- moved J4 232.5 mm to (253.5, 268.0), turned to -90 degrees
- moved U2 211.1 mm to (121.2, 272.5)
- moved U1 179.3 mm to (315.9, 159.9), turned to -90 degrees
- moved R1 138.9 mm to (255.8, 81.8)
- moved U3 132.6 mm to (247.4, 82.9)
- moved D7 132.0 mm to (251.8, 81.8)
- moved R4 130.6 mm to (268.6, 85.6)
- moved R16 127.5 mm to (235.6, 100.3), turned to 180 degrees
- moved R2 127.0 mm to (272.8, 81.8)
- moved D1 125.3 mm to (251.8, 84.4)
- moved C5 117.8 mm to (138.2, 197.1), turned to 0 degrees
- moved C1 115.5 mm to (259.8, 81.8)
- moved R12 114.1 mm to (250.9, 87.0)
- moved R17 114.1 mm to (250.9, 89.5)
- moved J2 112.8 mm to (82.0, 272.3), turned to 0 degrees
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Connections:
- C1 pad 1: Net-(C1-Pad1) -> /ChargeController/V_{in}_Sense
- C1 pad 2: /N -> Earth
- C10 pad 1: /N -> /V_{REG}
- C10 pad 2: Net-(C10-Pad2) -> Earth
- C12 pad 1: /V_{REG} -> /ChargeController/I_{in}Sense
- C13 pad 1: /V_{DC} -> /ChargeController/I_{in}Sense
- C2 pad 1: /L1 -> /ChargeController/V_{BATT}_Sense
- C2 pad 2: Net-(C2-Pad2) -> Earth
- C3 pad 1: /V_{DC} -> /ChargeController/I_{in}Sense
- C4 pad 1: /V_{DC} -> /ChargeController/I_{in}Sense
- C5 pad 1: Net-(C5-Pad1) -> /ChargeController/I_{in}Sense
- C5 pad 2: /L1 -> Earth
- C8 pad 1: Net-(C8-Pad1) -> /V_{REG}
- C8 pad 2: /ChargeController/V_{in}- -> Earth
- C9 pad 1: /V_{DC} -> /ChargeController/I_{in}Sense
- D1 pad 1: /V_{DC} -> /ChargeController/V_{BATT}_Sense
- D1 pad 2: Net-(C1-Pad1) -> Earth
- J1 pad 1: /N -> /L1
- J4 pad 11: /CAN Transiever/GND -> Earth
- J4 pad 9: /CAN Transiever/GND -> Earth
- L1 pad 1: Net-(L1-Pad1) -> /DC-DC Converter/L+
- L1 pad 2: Net-(L1-Pad2) -> /DC-DC Converter/L-
- Q1 pad 1: Net-(C1-Pad1) -> /FilteredRectifier/PHG2
- Q1 pad 2: /L1 -> /FilteredRectifier/PHS2
- Q1 pad 3: /V_{DC} -> /ChargeController/I_{in}Sense
- Q2 pad 1: Net-(C2-Pad2) -> /FilteredRectifier/PHG1
- Q2 pad 2: /N -> /FilteredRectifier/PHS1
- Q2 pad 3: /V_{DC} -> /FilteredRectifier/PHS2
- Q3 pad 1: Net-(C5-Pad1) -> /FilteredRectifier/PHG0
- Q3 pad 2: Earth -> /L1
- Q3 pad 3: /N -> /FilteredRectifier/PHS1
- Q4 pad 1: Net-(C10-Pad2) -> /FilteredRectifier/NLG2
- Q4 pad 2: Earth -> /FilteredRectifier/NLS2
- Q4 pad 3: /L1 -> /N
- Q5 pad 1: unconnected-(Q5-Pad1) -> /DC-DC Converter/BUCK_SG2
- Q5 pad 2: Net-(L1-Pad1) -> /DC-DC Converter/BUCK_SS2
- Q6 pad 1: unconnected-(Q6-Pad1) -> /DC-DC Converter/BUCK_DG0
- Q6 pad 3: Net-(L1-Pad1) -> /DC-DC Converter/BUCK_DS1
- Q7 pad 1: unconnected-(Q7-Pad1) -> /DC-DC Converter/BOOST_SG0
- Q7 pad 3: Net-(L1-Pad2) -> /DC-DC Converter/BOOST_SS1
- Q8 pad 2: /V_{BATT} -> /ChargeController/I_{Sense}+
- Q8 pad 3: Net-(Q8-Pad3) -> /V_{REG}
- Q9 pad 1: unconnected-(Q9-Pad1) -> /DC-DC Converter/BOOST_DG0
- Q9 pad 2: Net-(L1-Pad2) -> /DC-DC Converter/L-
- Q9 pad 3: /V_{REG} -> /DC-DC Converter/BOOST_DS1
- R1 pad 1: Net-(C1-Pad1) -> /ChargeController/V_{BATT}_Sense
- R1 pad 2: /N -> Earth
- R11 pad 1: Net-(Q8-Pad3) -> /V_{REG}
- R16 pad 1: Net-(R16-Pad1) -> Earth
- R16 pad 2: Net-(R16-Pad2) -> Net-(C11-Pad1)
- R17 pad 2: Net-(R17-Pad2) -> /ChargeController/V_{BATT}_Sense
- R18 pad 1: Net-(R17-Pad2) -> Net-(C11-Pad2)
- R18 pad 2: Earth -> /ChargeController/I_{BATT}_Sense
- R2 pad 2: Net-(C2-Pad2) -> Net-(R3-Pad1)
- R4 pad 1: /N -> Net-(R3-Pad2)
- R4 pad 2: Net-(C10-Pad2) -> /N
- R8 pad 1: /V_{DC} -> Net-(IC4-Pad7)
- R8 pad 2: Net-(C8-Pad1) -> /DC-DC Converter/BUCK_DG1
- U1 pad 1: /CAN Transiever/VCC -> +3V3
- U1 pad 4: /CAN Transiever/GND -> Earth
- U2 pad 1: unconnected-(U2-Pad1) -> /ChargeController/SWITCH
- U2 pad 11: unconnected-(U2-Pad11) -> /ChargeController/I_MAX
- U2 pad 12: unconnected-(U2-Pad12) -> /ChargeController/START/~{STOP}
- U2 pad 13: unconnected-(U2-Pad13) -> /ChargeController/BOOST/~{BUCK}
- U2 pad 15: /ChargeController/Buck_CTL -> unconnected-(U2-Pad15)
- U2 pad 18: /ChargeController/SWIM_DATA -> /ChargeController/SWIM
- U2 pad 19: unconnected-(U2-Pad19) -> /ChargeController/I_{BATT}_Sense
- U2 pad 2: unconnected-(U2-Pad2) -> /CAN Transiever/TXD
- U2 pad 20: unconnected-(U2-Pad20) -> /ChargeController/V_{BATT}_Sense
- U2 pad 3: Net-(R16-Pad1) -> /CAN Transiever/RXD
- U2 pad 4: unconnected-(U2-Pad4) -> /ChargeController/~{RST}
- U2 pad 8: unconnected-(U2-Pad8) -> Net-(C17-Pad1)
- U2 pad 9: unconnected-(U2-Pad9) -> +3V3
- U3 pad 1: unconnected-(U3-Pad1) -> /ChargeController/I_{BATT}_Sense
- U3 pad 2: unconnected-(U3-Pad2) -> Earth
- U3 pad 5: unconnected-(U3-Pad5) -> +3V3
- U4 pad 1: unconnected-(U4-Pad1) -> /FilteredRectifier/FORWARD
- U4 pad 2: unconnected-(U4-Pad2) -> Earth
- U4 pad 3: unconnected-(U4-Pad3) -> Net-(R3-Pad1)
- U4 pad 4: unconnected-(U4-Pad4) -> Net-(R3-Pad2)
- U4 pad 5: unconnected-(U4-Pad5) -> +3V3
Routing:
- net /ChargeController/~{RST}: track 0.00 -> 21.4 mm
- net /ChargeController/SWIM: track 0.00 -> 17.2 mm
- net +3V3: track 0.00 -> 5.08 mm
- net Net-(C8-Pad1): track 4.16 -> 0.00 mm
- net Net-(U2-Pad6): track 0.00 -> 3.85 mm
- net Net-(U2-Pad5): track 0.00 -> 3.85 mm
- net /ChargeController/V_{in}-: track 3.32 -> 0.00 mm
- net /CAN Transiever/CAN_VCC: track 0.00 -> 1.83 mm
- net /CAN Transiever/CAN_GND: track 0.00 -> 1.19 mm
- net /V_{REG}: vias 0 -> 20
- net /V_{DC}: vias 0 -> 20
- net /DC-DC Converter/L-: vias 0 -> 192
- net /DC-DC Converter/L+: vias 0 -> 195
- net /DC-DC Converter/BUCK_SS2: vias 0 -> 20
- net /DC-DC Converter/BUCK_SS1: vias 0 -> 20
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- added copper zone on B.Cu, net /ChargeController/I_{in}Sense
- added copper zone on F.Cu, net /ChargeController/I_{in}Sense
- added copper zone on B.Cu, net /DC-DC Converter/BOOST_DS1
- added copper zone on F.Cu, net /DC-DC Converter/BOOST_DS1
- added copper zone on B.Cu, net /DC-DC Converter/BOOST_DS2
- added copper zone on F.Cu, net /DC-DC Converter/BOOST_DS2
- added copper zone on B.Cu, net /DC-DC Converter/BOOST_SS1
- added copper zone on F.Cu, net /DC-DC Converter/BOOST_SS1
- added copper zone on B.Cu, net /DC-DC Converter/BOOST_SS2
- added copper zone on F.Cu, net /DC-DC Converter/BOOST_SS2
- added copper zone on B.Cu, net /DC-DC Converter/BUCK_DS1
- added copper zone on F.Cu, net /DC-DC Converter/BUCK_DS1
- added copper zone on B.Cu, net /DC-DC Converter/BUCK_DS2
- added copper zone on F.Cu, net /DC-DC Converter/BUCK_DS2
- added copper zone on B.Cu, net /DC-DC Converter/BUCK_SS1
- added copper zone on F.Cu, net /DC-DC Converter/BUCK_SS1
- added copper zone on B.Cu, net /DC-DC Converter/BUCK_SS2
- added copper zone on F.Cu, net /DC-DC Converter/BUCK_SS2
- added copper zone on B.Cu, net /DC-DC Converter/L+
- added copper zone on F.Cu, net /DC-DC Converter/L+
- added copper zone on B.Cu, net /DC-DC Converter/L-
- added copper zone on F.Cu, net /DC-DC Converter/L-
- added copper zone on B.Cu, net /FilteredRectifier/NHS1
- added copper zone on B.Cu, net /FilteredRectifier/NHS2
- added copper zone on B.Cu, net /FilteredRectifier/NLS1
- added copper zone on B.Cu, net /FilteredRectifier/NLS2
- added copper zone on B.Cu, net /FilteredRectifier/PHS1
- added copper zone on B.Cu, net /FilteredRectifier/PHS2
- added copper zone on B.Cu, net /FilteredRectifier/PLS1
- added copper zone on B.Cu, net /FilteredRectifier/PLS2
- added copper zone on B.Cu, net /L1
- added copper zone on B.Cu, net /N
- added copper zone on B.Cu, net /V_{DC}
- added copper zone on F.Cu, net /V_{DC}
- added copper zone on B.Cu, net /V_{REG}
- added copper zone on F.Cu, net /V_{REG}
- added copper zone on B.Cu, net Earth
Other:
- board size 193 x 99.1 mm -> 181.6 x 131.8 mm
- board text added: "Q6"

Commit message: Updated Charger and MC
Parts:
- removed C11: C_Small, Capacitor_SMD:C_0603_1608Metric
- removed IC10, IC11, IC12, IC13, IC5, IC6, IC7, IC8, IC9: 1EDI60N12AFXUMA1, SamacSys_Parts:SOIC127P600X175-8N
- removed J2: Conn_01x03, Connector_PinHeader_2.54mm:PinHeader_1x03_P2.54mm_Vertical
- removed J4: RJ45_LED, Connector_RJ:RJ45_Amphenol_RJHSE538X
- removed J5: Conn_01x02, Connector_PinHeader_2.54mm:PinHeader_1x02_P2.54mm_Vertical
- removed J6: Conn_01x01_Female, Connector:Banana_Jack_1Pin
- removed Q12, Q13, Q14, Q15, Q16, Q17, Q18, Q19, Q20, Q21, Q22, Q23, Q24, Q25, Q26: IPT015N10N5, Package_TO_SOT_SMD:Infineon_PG-HSOF-8-1
- removed the R14 at (246.9, 86.4)
- removed the R14 at (298.1, 82.6)
- removed the R15 at (246.9, 88.9)
- removed the R15 at (298.1, 80.1)
- removed R2: R_US, Resistor_SMD:R_0603_1608Metric
- removed the R7 at (284.5, 82.3)
- removed the R7 at (286.0, 142.2)
- removed U1: ISO1050DUB, Package_SO:SOP-8_6.62x9.15mm_P2.54mm
- removed U3: LMH6609MF, Package_TO_SOT_SMD:SOT-23-5
- removed U4: MCP6L01x-xLT, Package_TO_SOT_SMD:SOT-353_SC-70-5
- added C24: 100uF, Capacitor_THT:CP_Radial_D16.0mm_P7.50mm, B.Cu at (230.2, 154.9)
- added C25: 100uF, Capacitor_THT:CP_Radial_D16.0mm_P7.50mm, B.Cu at (230.2, 172.1)
- added C26: 100uF, Capacitor_THT:CP_Radial_D16.0mm_P7.50mm, B.Cu at (141.8, 156.2)
- added C27: 100uF, Capacitor_THT:CP_Radial_D16.0mm_P7.50mm, B.Cu at (141.8, 173.2)
- added L2: L, Inductor_THT:L_Toroid_Vertical_L22.4mm_W10.2mm_P7.90mm_Vishay_TJ4, F.Cu at (190.4, 123.2)
- added L3: L, Inductor_THT:L_Toroid_Vertical_L22.4mm_W10.2mm_P7.90mm_Vishay_TJ4, F.Cu at (190.5, 147.3)
- added R13: 10, Resistor_SMD:R_1206_3216Metric, F.Cu at (134.0, 125.7)
- added R14: 10, Resistor_SMD:R_1206_3216Metric, F.Cu at (134.0, 171.4)
- added R15: 10, Resistor_SMD:R_1206_3216Metric, F.Cu at (134.0, 168.9)
- added R5: 10, Resistor_SMD:R_1206_3216Metric, F.Cu at (134.0, 176.5)
- added R6: 10, Resistor_SMD:R_1206_3216Metric, F.Cu at (134.0, 118.1)
- added R7: .1m, Resistor_SMD:R_4020_10251Metric, F.Cu at (247.4, 173.5)
- added R9: 10, Resistor_SMD:R_1206_3216Metric, F.Cu at (134.0, 122.9)
- C10, C12, C13, C14, C15, C16, C3, C4, C5, C6, C8, C9: moved to B.Cu
- IC2, IC3, IC4: value 1EDI60N12AFXUMA1 -> STDRIVEG600TR; footprint SamacSys_Parts:SOIC127P600X175-8N -> SamacSys_Parts:SOIC127P600X175-16N
- J1: value Conn_01x01_Female -> Conn_01x02; footprint Connector:Banana_Jack_1Pin -> Connector:Banana_Jack_2Pin
- L1: footprint Inductor_THT:L_Toroid_Vertical_L67.6mm_W36.1mm_P31.80mm_Vishay_TJ9 -> Inductor_THT:L_Toroid_Vertical_L22.4mm_W10.2mm_P7.90mm_Vishay_TJ4
- Q1, Q3: value IPT015N10N5 -> BS170; footprint Package_TO_SOT_SMD:Infineon_PG-HSOF-8-1 -> Package_TO_SOT_THT:TO-92_Inline; moved to F.Cu
- Q10, Q11, Q2, Q6, Q8, Q9: value IPT015N10N5 -> Q_NMOS_GDS; footprint Package_TO_SOT_SMD:Infineon_PG-HSOF-8-1 -> Package_TO_SOT_SMD:TO-263-3_TabPin2; moved to F.Cu
- Q4: value IPT015N10N5 -> STB15N80K5; footprint Package_TO_SOT_SMD:Infineon_PG-HSOF-8-1 -> Package_TO_SOT_SMD:SOT-23; moved to F.Cu
- Q5, Q7: value IPT015N10N5 -> Q_NMOS_GDS; footprint Package_TO_SOT_SMD:Infineon_PG-HSOF-8-1 -> Package_TO_SOT_SMD:TO-263-3_TabPin2
- R18: value 99k -> R_US
- R4: value R_US -> 10; footprint Resistor_SMD:R_0603_1608Metric -> Resistor_SMD:R_1206_3216Metric
- R8: value R_Small_US -> 10
- moved R8 215.9 mm to (134.0, 115.6)
- moved Q11 197.8 mm to (260.4, 120.7), turned to 180 degrees
- moved Q10 175.2 mm to (242.6, 120.7), turned to 180 degrees
- moved U2 169.9 mm to (245.9, 157.2), turned to 90 degrees
- moved J7 169.7 mm to (242.1, 167.4)
- moved R4 163.8 mm to (134.0, 179.1)
- moved R1 147.9 mm to (252.8, 229.7)
- moved R18 137.1 mm to (148.6, 208.3), turned to 0 degrees
- moved R16 136.1 mm to (152.6, 208.3), turned to 0 degrees
- moved C14 128.2 mm to (230.2, 137.8), turned to 180 degrees
- moved C15 128.2 mm to (230.2, 120.7), turned to 180 degrees
- moved C12 126.4 mm to (141.8, 139.1)
- moved C1 119.8 mm to (231.3, 198.2)
- moved C2 119.8 mm to (231.3, 200.7)
- moved R10 117.4 mm to (227.3, 198.2)
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Connections:
- net /DC-DC Converter/BOOST_DG0 renamed /DC-DC Converter/G_DIODE
- C1 pad 2: Earth -> /ChargeController/GND
- C10 pad 2: Earth -> /ChargeController/GND
- C12 pad 1: /ChargeController/I_{in}Sense -> /V_{DC}
- C12 pad 2: Earth -> /ChargeController/GND
- C13 pad 1: /ChargeController/I_{in}Sense -> /V_{DC}
- C13 pad 2: Earth -> /ChargeController/GND
- C14 pad 2: Earth -> /ChargeController/GND
- C15 pad 2: Earth -> /ChargeController/GND
- C16 pad 2: Earth -> /ChargeController/GND
- C17 pad 2: Earth -> /ChargeController/GND
- C3 pad 1: /ChargeController/I_{in}Sense -> /V_{DC}
- C3 pad 2: Earth -> /ChargeController/GND
- C4 pad 1: /ChargeController/I_{in}Sense -> /V_{DC}
- C4 pad 2: Earth -> /ChargeController/GND
- C5 pad 1: /ChargeController/I_{in}Sense -> /V_{DC}
- C5 pad 2: Earth -> /ChargeController/GND
- C6 pad 2: Earth -> /ChargeController/GND
- C8 pad 2: Earth -> /ChargeController/GND
- C9 pad 1: /ChargeController/I_{in}Sense -> /V_{DC}
- C9 pad 2: Earth -> /ChargeController/GND
- D7 pad 2: Earth -> /ChargeController/GND
- IC1 pad 1: Earth -> /ChargeController/GND
- IC1 pad 2: Earth -> /ChargeController/GND
- IC2 pad 1: /DC-DC Converter/DC-DC Converter Gate Driver/3V3 -> /FilteredRectifier/NEG_ON
- IC2 pad 2: unconnected-(IC2-Pad2) -> +12V
- IC2 pad 3: Earth -> /FilteredRectifier/POS_ON
- IC2 pad 4: Earth -> +12V
- IC2 pad 5: +12V -> Net-(C7-Pad1)
- IC2 pad 7: unconnected-(IC2-Pad7) -> /FilteredRectifier/DGND
- IC3 pad 1: /DC-DC Converter/DC-DC Converter Gate Driver/3V3 -> /FilteredRectifier/POS_ON
- IC3 pad 2: unconnected-(IC3-Pad2) -> +12V
- IC3 pad 3: Earth -> /FilteredRectifier/NEG_ON
- IC3 pad 4: Earth -> +12V
- IC3 pad 5: +12V -> Net-(C19-Pad1)
- IC3 pad 7: unconnected-(IC3-Pad7) -> /FilteredRectifier/DGND
- IC4 pad 1: /DC-DC Converter/DC-DC Converter Gate Driver/3V3 -> /ChargeController/SWITCH
- IC4 pad 2: /DC-DC Converter/DC-DC Converter Gate Driver/BUCK_DIODE_EN -> +12V
- IC4 pad 3: Earth -> /DC-DC Converter/~{SWITCH}
- IC4 pad 4: Earth -> +12V
- IC4 pad 5: +12V -> Net-(C22-Pad1)
- IC4 pad 6: Net-(IC4-Pad6) -> unconnected-(IC4-Pad6)
- IC4 pad 7: Net-(IC4-Pad7) -> Earth
- J1 pad 1: /L1 -> /N
- J7 pad 3: Earth -> /ChargeController/GND
- J7 pad 4: Earth -> /ChargeController/GND
- L1 pad 2: /DC-DC Converter/L- -> /V_{REG}
- Q1 pad 1: /FilteredRectifier/PHG2 -> /FilteredRectifier/POS_ON
- Q1 pad 2: /FilteredRectifier/PHS2 -> unconnected-(Q1-Pad2)
- Q1 pad 3: /ChargeController/I_{in}Sense -> Net-(Q1-Pad3)
- Q10 pad 1: /FilteredRectifier/PLG2 -> unconnected-(Q10-Pad1)
- Q10 pad 2: /FilteredRectifier/PLS2 -> /V_{REG}
- Q10 pad 3: /L1 -> Net-(Q10-Pad3)
- Q11 pad 1: /FilteredRectifier/PLG1 -> unconnected-(Q11-Pad1)
- Q11 pad 2: /FilteredRectifier/PLS1 -> /V_{BATT}
- Q11 pad 3: /FilteredRectifier/PLS2 -> Net-(Q10-Pad3)
- Q2 pad 1: /FilteredRectifier/PHG1 -> /FilteredRectifier/PHG
- Q2 pad 2: /FilteredRectifier/PHS1 -> /V_{DC}
- Q2 pad 3: /FilteredRectifier/PHS2 -> /L1
- Q3 pad 1: /FilteredRectifier/PHG0 -> /FilteredRectifier/NEG_ON
- Q3 pad 2: /L1 -> /FilteredRectifier/POS_ON
- Q3 pad 3: /FilteredRectifier/PHS1 -> Net-(Q1-Pad3)
- Q4 pad 1: /FilteredRectifier/NLG2 -> /ChargeController/SWITCH
- Q4 pad 2: /FilteredRectifier/NLS2 -> /DC-DC Converter/~{SWITCH}
- Q4 pad 3: /N -> Earth
- Q5 pad 1: /DC-DC Converter/BUCK_SG2 -> /FilteredRectifier/PLG
- Q5 pad 2: /DC-DC Converter/BUCK_SS2 -> /L1
- Q5 pad 3: /V_{DC} -> /ChargeController/GND
- Q6 pad 1: /DC-DC Converter/BUCK_DG0 -> /FilteredRectifier/NHG
- Q6 pad 2: Earth -> /V_{DC}
- Q6 pad 3: /DC-DC Converter/BUCK_DS1 -> /N
- Q7 pad 1: /DC-DC Converter/BOOST_SG0 -> /FilteredRectifier/NLG
- Q7 pad 2: Earth -> /N
- Q7 pad 3: /DC-DC Converter/BOOST_SS1 -> /ChargeController/GND
- Q8 pad 1: unconnected-(Q8-Pad1) -> /DC-DC Converter/G_SWITCH
- Q8 pad 2: /ChargeController/I_{Sense}+ -> /V_{DC}
- Q8 pad 3: /V_{REG} -> /DC-DC Converter/L+
- Q9 pad 2: /DC-DC Converter/L- -> /DC-DC Converter/L+
- Q9 pad 3: /DC-DC Converter/BOOST_DS1 -> /ChargeController/GND
- R12 pad 2: Earth -> /ChargeController/GND
- R16 pad 1: Earth -> +3V3
- R16 pad 2: Net-(C11-Pad1) -> /FilteredRectifier/POS_ON
- R18 pad 1: Net-(C11-Pad2) -> +3V3
- R18 pad 2: /ChargeController/I_{BATT}_Sense -> /FilteredRectifier/NEG_ON
- R4 pad 1: Net-(R3-Pad2) -> /FilteredRectifier/NHG
- R4 pad 2: /N -> Net-(IC2-Pad15)
- R8 pad 1: Net-(IC4-Pad7) -> /FilteredRectifier/PLG
- R8 pad 2: /DC-DC Converter/BUCK_DG1 -> Net-(IC2-Pad10)
- U2 pad 11: /ChargeController/I_MAX -> unconnected-(U2-Pad11)
- U2 pad 2: /CAN Transiever/TXD -> unconnected-(U2-Pad2)
- U2 pad 3: /CAN Transiever/RXD -> unconnected-(U2-Pad3)
- U2 pad 7: Earth -> /ChargeController/GND
- Y1 pad 2: Earth -> /ChargeController/GND
Routing:
- net Net-(IC2-Pad10): track 0.00 -> 49.4 mm
- net Net-(IC3-Pad11): track 0.00 -> 48.1 mm
- net Net-(IC2-Pad11): track 0.00 -> 47.1 mm
- net Net-(IC3-Pad10): track 0.00 -> 46.1 mm
- net Net-(IC2-Pad15): track 0.00 -> 34.8 mm
- net Net-(IC2-Pad14): track 0.00 -> 31.4 mm
- net Net-(IC3-Pad15): track 0.00 -> 26.2 mm
- net Net-(IC3-Pad14): track 0.00 -> 20.3 mm
- net /ChargeController/~{RST}: track 21.4 -> 8.47 mm
- net /ChargeController/GND: track 0.00 -> 8.23 mm
- net /ChargeController/SWIM: track 17.2 -> 25.0 mm
- net /FilteredRectifier/PLG: track 0.00 -> 7.19 mm, vias 0 -> 1
- net /FilteredRectifier/NLG: track 0.00 -> 7.18 mm, vias 0 -> 1
- net /FilteredRectifier/PHG: track 0.00 -> 7.12 mm
- net /FilteredRectifier/NHG: track 0.00 -> 6.77 mm
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- removed copper zone on B.Cu, net /ChargeController/I_{in}Sense
- removed copper zone on F.Cu, net /ChargeController/I_{in}Sense
- removed copper zone on B.Cu, net /DC-DC Converter/BOOST_DS1
- removed copper zone on F.Cu, net /DC-DC Converter/BOOST_DS1
- removed copper zone on B.Cu, net /DC-DC Converter/BOOST_DS2
- removed copper zone on F.Cu, net /DC-DC Converter/BOOST_DS2
- removed copper zone on B.Cu, net /DC-DC Converter/BOOST_SS1
- removed copper zone on F.Cu, net /DC-DC Converter/BOOST_SS1
- removed copper zone on B.Cu, net /DC-DC Converter/BOOST_SS2
- removed copper zone on F.Cu, net /DC-DC Converter/BOOST_SS2
- removed copper zone on B.Cu, net /DC-DC Converter/BUCK_DS1
- removed copper zone on F.Cu, net /DC-DC Converter/BUCK_DS1
- removed copper zone on B.Cu, net /DC-DC Converter/BUCK_DS2
- removed copper zone on F.Cu, net /DC-DC Converter/BUCK_DS2
- removed copper zone on B.Cu, net /DC-DC Converter/BUCK_SS1
- removed copper zone on F.Cu, net /DC-DC Converter/BUCK_SS1
- removed copper zone on B.Cu, net /DC-DC Converter/BUCK_SS2
- removed copper zone on F.Cu, net /DC-DC Converter/BUCK_SS2
- removed copper zone on B.Cu, net /DC-DC Converter/L+
- removed copper zone on F.Cu, net /DC-DC Converter/L+
- removed copper zone on B.Cu, net /DC-DC Converter/L-
- removed copper zone on F.Cu, net /DC-DC Converter/L-
- removed copper zone on B.Cu, net /FilteredRectifier/NHS1
- removed copper zone on B.Cu, net /FilteredRectifier/NHS2
- removed copper zone on B.Cu, net /FilteredRectifier/NLS1
- removed copper zone on B.Cu, net /FilteredRectifier/NLS2
- removed copper zone on B.Cu, net /FilteredRectifier/PHS1
- removed copper zone on B.Cu, net /FilteredRectifier/PHS2
- removed copper zone on B.Cu, net /FilteredRectifier/PLS1
- removed copper zone on B.Cu, net /FilteredRectifier/PLS2
- removed copper zone on B.Cu, net /L1
- removed copper zone on B.Cu, net /N
- removed copper zone on B.Cu, net /V_{DC}
- removed copper zone on F.Cu, net /V_{DC}
- removed copper zone on B.Cu, net /V_{REG}
- removed copper zone on F.Cu, net /V_{REG}
- removed copper zone on B.Cu, net Earth
- removed copper zone on F.Cu, net Earth
Other:
- board outline removed
- board text removed: "Q6"
