File: OpenCharger/ChargeController.kicad_sch (KiCad schematic)
At the start: 16 parts, among them Q8 IPT015N10N5, U2 STM8AF6223A, U3 LMH6609MF, U5 LMH6609MF, Y1 Resonator_Small

Commit message: updated
Parts:
- removed C11: C_Small, Capacitor_SMD:C_0603_1608Metric, symbol Device:C_Small
- removed R13, R14, R15, R16, R18: R_US, Resistor_SMD:R_0603_1608Metric, symbol Device:R_US
- removed U3, U5: LMH6609MF, Package_TO_SOT_SMD:SOT-23-5, symbol Amplifier_Operational:LMH6609MF
- added C1, C17, C2: C, Capacitor_SMD:C_0603_1608Metric, symbol Device:C
- added C11, C18: C, symbol Device:C
- added D1: 5V, Diode_SMD:D_0603_1608Metric, symbol Device:D_Zener
- added IC1: INA211CQDCKRQ1, SOT65P210X110-6N, symbol SamacSys_Parts:INA211CQDCKRQ1
- added J7: Conn_02x05_Odd_Even, Connector_PinHeader_2.54mm:PinHeader_2x05_P2.54mm_Vertical, symbol Connector_Generic:Conn_02x05_Odd_Even
- added Q26: IPT015N10N5, Package_TO_SOT_SMD:Infineon_PG-HSOF-8-1, symbol Transistor_FET:IPT015N10N5
- added R1: 1k, Resistor_SMD:R_0603_1608Metric, symbol Device:R_US
- added R10: 10k, Resistor_SMD:R_0603_1608Metric, symbol Device:R_US
- R17: value R_US -> 99k
- R7: value R_Small -> .1m
Connections:
- net V_{BATT}+: now also R7.2, IC1.5 (IN-); no longer Q8.2 (S)
- net V_{BATT}-: now also C1.2, C11.2, C17.2, C18.2, C2.2, D1.2 (A), IC1.1 (REF), IC1.2 (GND), J7.3 (Pin_3), J7.4 (Pin_4), R1.2
- net V_{in}+: now also Q8.3 (D), R11.1, Q26.3 (D); no longer R7.1
- net V_{in}_Sense: now also C1.1
- net V_{BATT}_Sense: now reaches R17.2
- net V_{BATT}_Sense: now also U2.20 (PD3), C2.1, D1.1 (K), R1.1
- net RXD: now reaches U2.3 (PD6)
- net SWITCH: now reaches U2.1 (PD4)
- net I_MAX: now reaches U2.11 (PB4)
- net START/~{STOP}: now reaches U2.12 (PB1)
- net BOOST/~{BUCK}: now reaches U2.13 (PB0)
- net I_{BATT}_Sense: now reaches U2.19 (PD2)
- net I_{BATT}_Sense: now also IC1.6 (OUT)
- net TXD: now reaches U2.2 (PD5)
- net ~{RST}: now reaches U2.4 (NRST)
- net ~{RST}: now also J7.1 (Pin_1), R10.2
- net at U2.8 (VCAP): now also C17.1
- net +3V3: now reaches U2.9 (VDD)
- net +3V3: now also C11.1, C18.1, IC1.3 (V+), J7.7 (Pin_7), J7.8 (Pin_8), R10.1
- net Buck_CTL: no longer names the net of U2.15 (PC5)
- net SWIM_DATA renamed SWIM
- net SWIM: now also J7.5 (Pin_5)
- new net I_{Sense}+: IC1.4 (IN+), Q26.2 (S), Q8.2 (S), R7.1
- no-connect marks 0 -> 4
Other:
- note added: "Current Sense Amp"
- note added: "Programming Connector"
- moved on the sheet: R7

Commit message: Updated Charger and MC
Parts:
- removed Q26, Q8: IPT015N10N5, Package_TO_SOT_SMD:Infineon_PG-HSOF-8-1, symbol Transistor_FET:IPT015N10N5
- added Q10, Q11: Q_NMOS_GDS, Package_TO_SOT_SMD:TO-263-3_TabPin2, symbol Device:Q_NMOS_GDS
Connections:
- net I_{Sense}+: no longer R7.1
- net V_{BATT}+: now also Q11.2 (D); no longer R7.2
- net V_{BATT}-: now also R7.2; no longer C1.2, C11.2, C17.2, C18.2, D7.2 (A), IC1.1 (REF), IC1.2 (GND), J7.3 (Pin_3), J7.4 (Pin_4), R12.2, U2.7 (VSS), Y1.2
- net V_{in}+: now also Q10.2 (D)
- net I_MAX: no longer names the net of U2.11 (PB4)
- net RXD: no longer names the net of U2.3 (PD6)
- net TXD: no longer names the net of U2.2 (PD5)
- new net: Q10.3 (S), Q11.3 (S)
- new net V_{in}-: C1.2, C11.2, C17.2, C18.2, D7.2 (A), IC1.1 (REF), IC1.2 (GND), J7.3 (Pin_3), J7.4 (Pin_4), R12.2, R7.1, U2.7 (VSS), Y1.2
Other:
- moved on the sheet: C11, C18, R7
