File: OpenCharger/ChargerInterface.kicad_sch (KiCad schematic)
At the start: 0 parts

Commit message: updated
Changed lines of the file:
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@@
 (kicad_sch (version 20210621) (generator eeschema)
   (paper "A4")
+  (hierarchical_label "I_MAX" (shape input) (at 199.39 85.09 0)
+    (effects (font (size 1.27 1.27)) (justify left))
+  )
   (hierarchical_label "PP" (shape input) (at 96.52 87.63 0)
     (effects (font (size 1.27 1.27)) (justify left))
   )
+  (hierarchical_label "START{slash}~{STOP}" (shape input) (at 195.58 78.74 0)
+    (effects (font (size 1.27 1.27)) (justify left))
+  )
