File: OpenMC/OpenMC.kicad_sch (KiCad schematic)
At the start: 0 parts

Commit message: Updated Charger and MC
Parts:
- added IC1: EFM8LB11F32E-C-QFN24, EFM8LB11F32EBQFN24R, symbol SamacSys_Parts:EFM8LB11F32E-C-QFN24
- added J3, J5: Conn_01x01_Female, Connector:Banana_Jack_1Pin, symbol Connector:Conn_01x01_Female
- added J4: Conn_01x06_Female, Connector_PinHeader_1.27mm:PinHeader_1x06_P1.27mm_Vertical, symbol Connector:Conn_01x06_Female
Connections:
- new net +BATT: J3.1 (Pin_1)
- new net BRAKE: IC1.10 (P2.0), J4.4 (Pin_4)
- new net COAST: IC1.9 (P2.1), J4.3 (Pin_3)
- new net EN: IC1.8 (P2.2), J4.2 (Pin_2)
- new net Earth: J5.1 (Pin_1)
- new net GND: IC1.15 (GND_2), IC1.25 (EP), IC1.3 (GND_1), J4.1 (Pin_1)
- new net PWM: IC1.11 (P1.6), J4.5 (Pin_5)
- new net RST: IC1.5 (RSTB_/_C2CK)
- new net VDD: IC1.4 (VDD_/_VIO), J4.6 (Pin_6)
Other:
- added sheet Left Driver FETs (DriverFETs.kicad_sch)
- added sheet Left Hall Sensors (HallSensors.kicad_sch)
- added sheet Right Driver FETs (DriverFETs.kicad_sch)
- added sheet Right Hall Sensors (HallSensors.kicad_sch)
