File: OpenMC/Controller.kicad_sch (KiCad schematic)
At the start: 1 part, among them IC1 EFM8BB31F32G-D-QSOP24R

Commit message: pcb work
Parts:
- removed IC1: EFM8BB31F32G-D-QSOP24R, symbol SamacSys_Parts:EFM8BB31F32G-D-QSOP24R
- added C10, C11, C12, C13, C9: 1uF, Capacitor_SMD:C_0603_1608Metric, symbol Device:C
- added IC1: ESP32-C3, QFN50P500X500X90-33N-D, symbol SamacSys_Parts:ESP32-C3
- added J8: 216990-0001, 2169900001, symbol SamacSys_Parts:216990-0001
- added U4: LM3480-3.3, Package_TO_SOT_SMD:SOT-23, symbol Regulator_Linear:LM3480-3.3
- added Y1: 40MHz, SamacSys_Parts:ABM12W300000MHZ6B1UT3, symbol Device:Crystal_GND24
Connections:
- net AH: now also IC1.15 (GPIO9)
- net AL: now also IC1.14 (GPIO8)
- net BH: now also IC1.13 (MTDO)
- net BL: now also IC1.12 (MTCK)
- net CS: now also IC1.21 (SPICS0)
- net GND: now also C10.2, C11.2, C12.2, C13.2, C9.2, IC1.33 (GND), J8.A1 (GND_1), J8.A12 (GND_2), J8.B1 (GND_3), J8.B12 (GND_4), J8.MH1, J8.MH2, J8.MH3, J8.MH4, U4.3 (GND), Y1.2, Y1.4
- net HALL_A: now also IC1.4 (XTAL_32K_P)
- net HALL_B: now also IC1.5 (XTAL_32K_N)
- net HALL_C: now also IC1.6 (GPIO2)
- net MISO: now also IC1.24 (SPIQ)
- net MOSI: now also IC1.23 (SPID)
- net SCLK: now also IC1.22 (SPICLK)
- new net: IC1.29 (XTAL_N), Y1.1
- new net: IC1.30 (XTAL_P), Y1.3
- new net 3V3: C10.1, C11.1, C12.1, C13.1, IC1.11 (VDD3P3_RTC), IC1.17 (VDD3P3_CPU), IC1.18 (VDD_SPI), IC1.2 (VDD3P3_1), IC1.3 (VDD3P3_2), IC1.31 (VDDA_1), IC1.32 (VDDA_2), U4.1 (VO)
- new net D+: IC1.26 (GPIO19), J8.A6 (DP1), J8.B6 (DP2)
- new net D-: IC1.25 (GPIO18), J8.A7 (DN1), J8.B7 (DN2)
- new net I_{SENSE}: IC1.8 (GPIO3)
- new net RST: IC1.7 (CHIP_EN)
- new net VBUS: C9.1, J8.A4 (VBUS_1), J8.A9 (VBUS_2), J8.B4 (VBUS_3), J8.B9 (VBUS_4), U4.2 (VI)
- new net V_{TEMP}: IC1.9 (MTMS)

Commit message: Updated PCB
Parts:
- added R11, R13, R14, R15, R5, R8: R_US, Resistor_SMD:R_0603_1608Metric, symbol Device:R_US
Connections:
- net AH: now also IC1.13 (MTDO); no longer IC1.15 (GPIO9)
- net AL: now also IC1.12 (MTCK); no longer IC1.14 (GPIO8)
- net BH: now also IC1.5 (XTAL_32K_N); no longer IC1.13 (MTDO)
- net BL: now also IC1.4 (XTAL_32K_P); no longer IC1.12 (MTCK)
- net CH: now also IC1.28 (U0TXD)
- net CL: now also IC1.27 (U0RXD)
- net HALL_A: now also IC1.16 (GPIO10), R13.2; no longer IC1.4 (XTAL_32K_P)
- net HALL_B: now also IC1.15 (GPIO9), R11.2; no longer IC1.5 (XTAL_32K_N)
- net HALL_C: now also IC1.14 (GPIO8), R8.2; no longer IC1.6 (GPIO2)
- net RST: now also IC1.6 (GPIO2), R5.2
- net I_{SENSE}A: now reaches IC1.10 (MTDI)
- net 3V3 renamed VDD
- net VDD: now also R11.1, R13.1, R14.1, R15.1, R5.1, R8.1
- net CS: no longer names the net of IC1.21 (SPICS0)
- net I_{SENSE} renamed I_{SENSE}B
- net MISO renamed SDA
- net SDA: now also R15.2
- net MOSI renamed SCL
- net SCL: now also R14.2
- net SCLK: no longer names the net of IC1.22 (SPICLK)
- net V_{TEMP} renamed I_{SENSE}C
Other:
- note added: "Debug Power Conversion"
- note added: "MCU"
- note added: "Pull Ups"
- note added: "USB Connector"
- moved on the sheet: C10, C11, C12, C13, C9, IC1, J8, U4, Y1
