File: OpenMC/CurrentSense.kicad_sch (KiCad schematic)
At the start: 1 part, among them IC4 INA186A4QDBVRQ1

Commit message: Updated PCB
Parts:
- renumbered IC4 to IC2
Changed lines of the file:
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@@
   (symbol (lib_id "SamacSys_Parts:INA186A4QDBVRQ1") (at 129.54 86.36 0)
     (in_bom yes) (on_board yes) (fields_autoplaced)
-    (property "Reference" "IC4" (id 0) (at 142.24 79.9043 0))
+    (property "Reference" "IC2" (id 0) (at 142.24 79.9043 0))
     (property "Value" "INA186A4QDBVRQ1" (id 1) (at 142.24 82.6794 0))
     (property "Footprint" "SOT95P280X145-5N" (id 2) (at 151.13 83.82 0)
