File: OpenMC/DriverFETs.kicad_sch (KiCad schematic)
At the start: 18 parts, among them J10 Conn_01x01_Female, J11 Conn_01x01_Female, J9 Conn_01x01_Female, Q13 BSC026N08NS5, Q14 BSC026N08NS5, Q15 BSC026N08NS5, Q16 BSC026N08NS5, Q17 BSC026N08NS5, Q18 BSC026N08NS5, Q19 BSC026N08NS5, Q20 BSC026N08NS5, Q21 BSC026N08NS5, Q22 BSC026N08NS5, Q23 BSC026N08NS5, Q24 BSC026N08NS5

Commit message: updates
Parts:
- removed J10, J11, J9: Conn_01x01_Female, Connector:Banana_Jack_1Pin, symbol Connector:Conn_01x01_Female
- R1: renamed from R4; footprint WSL36371L000DEA -> (none)
- R2: renamed from R5; footprint WSL36371L000DEA -> (none)
- R3: renamed from R6; footprint WSL36371L000DEA -> (none)
- renumbered Q13 to Q1, Q22 to Q10, Q23 to Q11, Q24 to Q12, Q14 to Q2, Q15 to Q3, Q16 to Q4, Q17 to Q5, Q18 to Q6, Q19 to Q7, Q20 to Q8, Q21 to Q9
Changed lines of the file:
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@@
-    (stroke (width 0) (type default) (color 0 0 0 0))
-  )
-  (wire (pts (xy 210.82 99.06) (xy 208.28 99.06))
     (stroke (width 0) (type default) (color 0 0 0 0))
   )
@@
     (stroke (width 0) (type default) (color 0 0 0 0))
   )
-  (wire (pts (xy 210.82 92.71) (xy 208.28 92.71))
-    (stroke (width 0) (type default) (color 0 0 0 0))
-  )
   (wire (pts (xy 111.76 78.74) (xy 111.76 76.2))
     (stroke (width 0) (type default) (color 0 0 0 0))
@@
     (stroke (width 0) (type default) (color 0 0 0 0))
   )
-  (wire (pts (xy 210.82 86.36) (xy 208.28 86.36))
-    (stroke (width 0) (type default) (color 0 0 0 0))
-  )
   (wire (pts (xy 93.98 106.68) (xy 102.87 106.68))
     (stroke (width 0) (type default) (color 0 0 0 0))
@@
     (effects (font (size 1.27 1.27)) (justify left bottom))
   )
-  (label "A" (at 208.28 86.36 0)
-    (effects (font (size 1.27 1.27)) (justify left bottom))
-  )
   (label "AL" (at 101.6 99.06 0)
     (effects (font (size 1.27 1.27)) (justify left bottom))
@@
     (effects (font (size 1.27 1.27)) (justify left bottom))
   )
-  (label "C" (at 208.28 99.06 0)
-    (effects (font (size 1.27 1.27)) (justify left bottom))
-  )
   (label "ISA" (at 97.79 106.68 0)
     (effects (font (size 1.27 1.27)) (justify left bottom))
@@
     (effects (font (size 1.27 1.27)) (justify left bottom))
   )
-  (label "B" (at 208.28 92.71 0)
-    (effects (font (size 1.27 1.27)) (justify left bottom))
-  )
   (label "B" (at 140.97 91.44 0)
     (effects (font (size 1.27 1.27)) (justify left bottom))
@@
     (effects (font (size 1.27 1.27)) (justify left bottom))
   )
+  (hierarchical_label "C" (shape input) (at 190.5 91.44 0)
+    (effects (font (size 1.27 1.27)) (justify left))
+  )
   (hierarchical_label "ISA+" (shape input) (at 80.01 110.49 180)
     (effects (font (size 1.27 1.27)) (justify right))
@@
     (effects (font (size 1.27 1.27)) (justify right))
   )
+  (hierarchical_label "A" (shape input) (at 111.76 91.44 0)
+    (effects (font (size 1.27 1.27)) (justify left))
+  )
   (hierarchical_label "ISB-" (shape input) (at 119.38 113.03 180)
     (effects (font (size 1.27 1.27)) (justify right))
@@
   (hierarchical_label "ISA-" (shape input) (at 80.01 113.03 180)
     (effects (font (size 1.27 1.27)) (justify right))
+  )
+  (hierarchical_label "B" (shape input) (at 151.13 91.44 0)
+    (effects (font (size 1.27 1.27)) (justify left))
   )
   (hierarchical_label "GND" (shape input) (at 88.9 116.84 180)
@@
   (symbol (lib_id "SamacSys_Parts:WSL36371L000DEA") (at 102.87 110.49 0) (mirror y)
     (in_bom yes) (on_board yes)
-    (property "Reference" "R4" (id 0) (at 86.36 106.68 0))
+    (property "Reference" "R1" (id 0) (at 86.36 106.68 0))
     (property "Value" "WSL36371L000DEA" (id 1) (at 113.03 113.03 0)
       (effects (font (size 1.27 1.27)) hide)
     )
-    (property "Footprint" "WSL36371L000DEA" (id 2) (at 83.82 107.95 0)
+    (property "Footprint" "" (id 2) (at 83.82 107.95 0)
       (effects (font (size 1.27 1.27)) (justify left) hide)
     )
@@
     (pin "L2")
   )
-  (symbol (lib_id "Connector:Conn_01x01_Female") (at 215.9 86.36 0)
-    (in_bom yes) (on_board yes) (fields_autoplaced)
-    (property "Reference" "J9" (id 0) (at 216.6112 85.4515 0)
-      (effects (font (size 1.27 1.27)) (justify left))
-    )
-    (property "Value" "Conn_01x01_Female" (id 1) (at 216.6112 88.2266 0)
-      (effects (font (size 1.27 1.27)) (justify left))
-    )
-    (property "Footprint" "Connector:Banana_Jack_1Pin" (id 2) (at 215.9 86.36 0)
-      (effects (font (size 1.27 1.27)) hide)
-    )
-    (property "Datasheet" "~" (id 3) (at 215.9 86.36 0)
-      (effects (font (size 1.27 1.27)) hide)
-    )
-    (pin "1")
-  )
   (symbol (lib_id "Transistor_FET:BSC026N08NS5") (at 130.81 99.06 0)
     (in_bom yes) (on_board yes) (fields_autoplaced)
-    (property "Reference" "Q18" (id 0) (at 136.017 98.1515 0)
+    (property "Reference" "Q6" (id 0) (at 136.017 98.1515 0)
       (effects (font (size 1.27 1.27)) (justify left))
     )
@@
     (pin "5")
   )
-  (symbol (lib_id "Connector:Conn_01x01_Female") (at 215.9 92.71 0)
-    (in_bom yes) (on_board yes) (fields_autoplaced)
-    (property "Reference" "J10" (id 0) (at 216.6112 91.8015 0)
-      (effects (font (size 1.27 1.27)) (justify left))
-    )
-    (property "Value" "Conn_01x01_Female" (id 1) (at 216.6112 94.5766 0)
-      (effects (font (size 1.27 1.27)) (justify left))
-    )
-    (property "Footprint" "Connector:Banana_Jack_1Pin" (id 2) (at 215.9 92.71 0)
-      (effects (font (size 1.27 1.27)) hide)
-    )
-    (property "Datasheet" "~" (id 3) (at 215.9 92.71 0)
-      (effects (font (size 1.27 1.27)) hide)
-    )
-    (pin "1")
-  )
-  (symbol (lib_id "Connector:Conn_01x01_Female") (at 215.9 99.06 0)
-    (in_bom yes) (on_board yes) (fields_autoplaced)
-    (property "Reference" "J11" (id 0) (at 216.6112 98.1515 0)
-      (effects (font (size 1.27 1.27)) (justify left))
-    )
-    (property "Value" "Conn_01x01_Female" (id 1) (at 216.6112 100.9266 0)
-      (effects (font (size 1.27 1.27)) (justify left))
-    )
-    (property "Footprint" "Connector:Banana_Jack_1Pin" (id 2) (at 215.9 99.06 0)
-      (effects (font (size 1.27 1.27)) hide)
-    )
-    (property "Datasheet" "~" (id 3) (at 215.9 99.06 0)
-      (effects (font (size 1.27 1.27)) hide)
-    )
-    (pin "1")
-  )
   (symbol (lib_id "Transistor_FET:BSC026N08NS5") (at 130.81 83.82 0)
     (in_bom yes) (on_board yes) (fields_autoplaced)
-    (property "Reference" "Q17" (id 0) (at 136.017 82.9115 0)
+    (property "Reference" "Q5" (id 0) (at 136.017 82.9115 0)
       (effects (font (size 1.27 1.27)) (justify left))
     )
@@
   (symbol (lib_id "Transistor_FET:BSC026N08NS5") (at 91.44 99.06 0)
     (in_bom yes) (on_board yes) (fields_autoplaced)
-    (property "Reference" "Q14" (id 0) (at 96.647 98.1515 0)
+    (property "Reference" "Q2" (id 0) (at 96.647 98.1515 0)
       (effects (font (size 1.27 1.27)) (justify left))
     )
@@
   (symbol (lib_id "Transistor_FET:BSC026N08NS5") (at 187.96 99.06 0)
     (in_bom yes) (on_board yes) (fields_autoplaced)
-    (property "Reference" "Q24" (id 0) (at 193.167 98.1515 0)
+    (property "Reference" "Q12" (id 0) (at 193.167 98.1515 0)
       (effects (font (size 1.27 1.27)) (justify left))
     )
@@
   (symbol (lib_id "SamacSys_Parts:WSL36371L000DEA") (at 181.61 110.49 0) (mirror y)
     (in_bom yes) (on_board yes)
-    (property "Reference" "R6" (id 0) (at 165.1 106.68 0))
+    (property "Reference" "R3" (id 0) (at 165.1 106.68 0))
     (property "Value" "WSL36371L000DEA" (id 1) (at 191.77 113.03 0)
       (effects (font (size 1.27 1.27)) hide)
     )
-    (property "Footprint" "WSL36371L000DEA" (id 2) (at 162.56 107.95 0)
+    (property "Footprint" "" (id 2) (at 162.56 107.95 0)
       (effects (font (size 1.27 1.27)) (justify left) hide)
     )
@@
   (symbol (lib_id "Transistor_FET:BSC026N08NS5") (at 168.91 83.82 0)
     (in_bom yes) (on_board yes) (fields_autoplaced)
-    (property "Reference" "Q21" (id 0) (at 174.117 82.9115 0)
+    (property "Reference" "Q9" (id 0) (at 174.117 82.9115 0)
       (effects (font (size 1.27 1.27)) (justify left))
     )
@@
   (symbol (lib_id "Transistor_FET:BSC026N08NS5") (at 109.22 99.06 0)
     (in_bom yes) (on_board yes) (fields_autoplaced)
-    (property "Reference" "Q16" (id 0) (at 114.427 98.1515 0)
+    (property "Reference" "Q4" (id 0) (at 114.427 98.1515 0)
       (effects (font (size 1.27 1.27)) (justify left))
     )
@@
   (symbol (lib_id "Transistor_FET:BSC026N08NS5") (at 148.59 83.82 0)
     (in_bom yes) (on_board yes) (fields_autoplaced)
-    (property "Reference" "Q19" (id 0) (at 153.797 82.9115 0)
+    (property "Reference" "Q7" (id 0) (at 153.797 82.9115 0)
       (effects (font (size 1.27 1.27)) (justify left))
     )
@@
   (symbol (lib_id "Transistor_FET:BSC026N08NS5") (at 109.22 83.82 0)
     (in_bom yes) (on_board yes) (fields_autoplaced)
-    (property "Reference" "Q15" (id 0) (at 114.427 82.9115 0)
+    (property "Reference" "Q3" (id 0) (at 114.427 82.9115 0)
       (effects (font (size 1.27 1.27)) (justify left))
     )
@@
   (symbol (lib_id "Transistor_FET:BSC026N08NS5") (at 148.59 99.06 0)
     (in_bom yes) (on_board yes) (fields_autoplaced)
-    (property "Reference" "Q20" (id 0) (at 153.797 98.1515 0)
+    (property "Reference" "Q8" (id 0) (at 153.797 98.1515 0)
       (effects (font (size 1.27 1.27)) (justify left))
     )
@@
   (symbol (lib_id "Transistor_FET:BSC026N08NS5") (at 168.91 99.06 0)
     (in_bom yes) (on_board yes) (fields_autoplaced)
-    (property "Reference" "Q22" (id 0) (at 174.117 98.1515 0)
+    (property "Reference" "Q10" (id 0) (at 174.117 98.1515 0)
       (effects (font (size 1.27 1.27)) (justify left))
     )
@@
   (symbol (lib_id "SamacSys_Parts:WSL36371L000DEA") (at 142.24 110.49 0) (mirror y)
     (in_bom yes) (on_board yes)
-    (property "Reference" "R5" (id 0) (at 125.73 106.68 0))
+    (property "Reference" "R2" (id 0) (at 125.73 106.68 0))
     (property "Value" "WSL36371L000DEA" (id 1) (at 152.4 113.03 0)
       (effects (font (size 1.27 1.27)) hide)
     )
-    (property "Footprint" "WSL36371L000DEA" (id 2) (at 123.19 107.95 0)
+    (property "Footprint" "" (id 2) (at 123.19 107.95 0)
       (effects (font (size 1.27 1.27)) (justify left) hide)
     )
@@
   (symbol (lib_id "Transistor_FET:BSC026N08NS5") (at 91.44 83.82 0)
     (in_bom yes) (on_board yes) (fields_autoplaced)
-    (property "Reference" "Q13" (id 0) (at 96.647 82.9115 0)
+    (property "Reference" "Q1" (id 0) (at 96.647 82.9115 0)
       (effects (font (size 1.27 1.27)) (justify left))
     )
@@
   (symbol (lib_id "Transistor_FET:BSC026N08NS5") (at 187.96 83.82 0)
     (in_bom yes) (on_board yes) (fields_autoplaced)
-    (property "Reference" "Q23" (id 0) (at 193.167 82.9115 0)
-      (effects (font (size 1.27 1.27)) (justify left))
-    )
+    (property "Reference" "Q11" (id 0) (at 193.167 82.9115 0)
+      (effects (font (size 1.27 1.27)) (justify left))
+    )

Commit message: pcb work
Parts:
- removed R1, R2, R3: WSL36371L000DEA, symbol SamacSys_Parts:WSL36371L000DEA
- added R1, R2, R3: PSR400ITQFL3L00, RESC10052X200N, symbol SamacSys_Parts:PSR400ITQFL3L00
- Q1, Q10, Q11, Q12, Q2, Q3, Q4, Q5, Q6, Q7, Q8, Q9: value BSC026N08NS5 -> SIR188DP; footprint Package_TO_SOT_SMD:TDSON-8-1 -> Package_SO:PowerPAK_SO-8_Single
Connections:
- net ISB is gone; now on net IS: Q6.1 (S), Q6.2 (S), Q6.3 (S), Q8.1 (S), Q8.2 (S), Q8.3 (S)
- net ISC is gone; now on net IS: Q10.1 (S), Q10.2 (S), Q10.3 (S), Q12.1 (S), Q12.2 (S), Q12.3 (S)
- net GND: now also R1.1, R2.1, R3.1
- net ISA renamed IS
- net IS: now also R1.2, R2.2, R3.2

Commit message: Updated PCB
Parts:
- removed R1, R2, R3: PSR400ITQFL3L00, RESC10052X200N, symbol SamacSys_Parts:PSR400ITQFL3L00
- added R1, R2, R3: WSLF25121L000FEB, RESC6430X38N, symbol SamacSys_Parts:WSLF25121L000FEB
Connections:
- net GND: now also R1.1, R2.1, R3.1
- removed net IS: Q10.1 (S), Q10.2 (S), Q10.3 (S), Q12.1 (S), Q12.2 (S), Q12.3 (S), Q2.1 (S), Q2.2 (S), Q2.3 (S), Q4.1 (S), Q4.2 (S), Q4.3 (S), Q6.1 (S), Q6.2 (S), Q6.3 (S), Q8.1 (S), Q8.2 (S), Q8.3 (S)
- new net ISA: Q2.1 (S), Q2.2 (S), Q2.3 (S), Q4.1 (S), Q4.2 (S), Q4.3 (S), R1.2
- new net ISB: Q6.1 (S), Q6.2 (S), Q6.3 (S), Q8.1 (S), Q8.2 (S), Q8.3 (S), R2.2
- new net ISC: Q10.1 (S), Q10.2 (S), Q10.3 (S), Q12.1 (S), Q12.2 (S), Q12.3 (S), R3.2
