File: OpenMC/GateDriver.kicad_sch (KiCad schematic)
At the start: 0 parts

Commit message: pcb work
Other:
- sheet Current Sense A renamed Current Sense Amp
- removed sheet Current Sense B
- removed sheet Current Sense C
- removed sheet VGen
Changed lines of the file:
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@@
     (stroke (width 0) (type default) (color 0 0 0 0))
   )
-  (hierarchical_label "ISB+" (shape input) (at 171.45 92.71 180)
-    (effects (font (size 1.27 1.27)) (justify right))
-  )
-  (hierarchical_label "3V3" (shape input) (at 171.45 113.03 180)
+  (hierarchical_label "V_{DRIVE}" (shape input) (at 115.57 66.04 180)
     (effects (font (size 1.27 1.27)) (justify right))
   )
@@
     (effects (font (size 1.27 1.27)) (justify left))
   )
-  (hierarchical_label "VBatt" (shape input) (at 86.36 67.31 180)
-    (effects (font (size 1.27 1.27)) (justify right))
-  )
-  (hierarchical_label "ISC+" (shape input) (at 171.45 116.84 180)
-    (effects (font (size 1.27 1.27)) (justify right))
+  (hierarchical_label "I_{SENSE}" (shape input) (at 205.74 91.44 0)
+    (effects (font (size 1.27 1.27)) (justify left))
   )
   (hierarchical_label "A" (shape input) (at 158.75 71.12 0)
     (effects (font (size 1.27 1.27)) (justify left))
   )
-  (hierarchical_label "IOUTA" (shape input) (at 190.5 68.58 0)
-    (effects (font (size 1.27 1.27)) (justify left))
-  )
-  (hierarchical_label "GND" (shape input) (at 171.45 123.19 180)
-    (effects (font (size 1.27 1.27)) (justify right))
-  )
-  (hierarchical_label "ISA+" (shape input) (at 171.45 69.85 180)
+  (hierarchical_label "IS" (shape input) (at 186.69 92.71 180)
     (effects (font (size 1.27 1.27)) (justify right))
   )
   (hierarchical_label "GCH" (shape input) (at 158.75 114.3 0)
-    (effects (font (size 1.27 1.27)) (justify left))
-  )
-  (hierarchical_label "GND" (shape input) (at 171.45 95.25 180)
-    (effects (font (size 1.27 1.27)) (justify right))
-  )
-  (hierarchical_label "3V3" (shape input) (at 115.57 68.58 0)
     (effects (font (size 1.27 1.27)) (justify left))
   )
@@
     (effects (font (size 1.27 1.27)) (justify right))
   )
-  (hierarchical_label "GND" (shape input) (at 171.45 99.06 180)
-    (effects (font (size 1.27 1.27)) (justify right))
-  )
   (hierarchical_label "CL" (shape input) (at 134.62 118.11 180)
     (effects (font (size 1.27 1.27)) (justify right))
   )
-  (hierarchical_label "3V3" (shape input) (at 171.45 88.9 180)
-    (effects (font (size 1.27 1.27)) (justify right))
-  )
-  (hierarchical_label "GND" (shape input) (at 171.45 72.39 180)
+  (hierarchical_label "GND" (shape input) (at 186.69 95.25 180)
     (effects (font (size 1.27 1.27)) (justify right))
   )
@@
     (effects (font (size 1.27 1.27)) (justify left))
   )
-  (hierarchical_label "GND" (shape input) (at 115.57 76.2 0)
-    (effects (font (size 1.27 1.27)) (justify left))
-  )
   (hierarchical_label "GND" (shape input) (at 134.62 121.92 180)
     (effects (font (size 1.27 1.27)) (justify right))
-  )
-  (hierarchical_label "IOUTC" (shape input) (at 190.5 115.57 0)
-    (effects (font (size 1.27 1.27)) (justify left))
   )
   (hierarchical_label "B" (shape input) (at 158.75 93.98 0)
     (effects (font (size 1.27 1.27)) (justify left))
   )
-  (hierarchical_label "GND" (shape input) (at 171.45 76.2 180)
-    (effects (font (size 1.27 1.27)) (justify right))
-  )
-  (hierarchical_label "3V3" (shape input) (at 171.45 66.04 180)
+  (hierarchical_label "GND" (shape input) (at 186.69 99.06 180)
     (effects (font (size 1.27 1.27)) (justify right))
   )
@@
     (effects (font (size 1.27 1.27)) (justify right))
   )
+  (hierarchical_label "VDD" (shape input) (at 186.69 88.9 180)
+    (effects (font (size 1.27 1.27)) (justify right))
+  )
   (hierarchical_label "CH" (shape input) (at 134.62 115.57 180)
     (effects (font (size 1.27 1.27)) (justify right))
   )
-  (hierarchical_label "IOUTB" (shape input) (at 190.5 91.44 0)
-    (effects (font (size 1.27 1.27)) (justify left))
-  )
-  (hierarchical_label "GND" (shape input) (at 171.45 119.38 180)
-    (effects (font (size 1.27 1.27)) (justify right))
-  )
-  (sheet (at 171.45 110.49) (size 19.05 15.24) (fields_autoplaced)
+  (sheet (at 186.69 86.36) (size 19.05 15.24) (fields_autoplaced)
     (stroke (width 0.1524) (type solid) (color 0 0 0 0))
     (fill (color 0 0 0 0.0000))
-    (property "Sheet name" "Current Sense C" (id 0) (at 171.45 109.7784 0)
+    (property "Sheet name" "Current Sense Amp" (id 0) (at 186.69 85.6484 0)
       (effects (font (size 1.27 1.27)) (justify left bottom))
     )
-    (property "Sheet file" "CurrentSense.kicad_sch" (id 1) (at 171.45 126.3146 0)
+    (property "Sheet file" "CurrentSense.kicad_sch" (id 1) (at 186.69 102.1846 0)
       (effects (font (size 1.27 1.27)) (justify left top))
     )
-    (pin "GND" input (at 171.45 123.19 180)
+    (pin "GND" input (at 186.69 99.06 180)
       (effects (font (size 1.27 1.27)) (justify left))
     )
-    (pin "IS-" input (at 171.45 119.38 180)
+    (pin "IS-" input (at 186.69 95.25 180)
       (effects (font (size 1.27 1.27)) (justify left))
     )
-    (pin "IS+" input (at 171.45 116.84 180)
+    (pin "IS+" input (at 186.69 92.71 180)
       (effects (font (size 1.27 1.27)) (justify left))
     )
-    (pin "IOUT" input (at 190.5 115.57 0)
+    (pin "IOUT" input (at 205.74 91.44 0)
       (effects (font (size 1.27 1.27)) (justify right))
     )
-    (pin "VDD" input (at 171.45 113.03 180)
-      (effects (font (size 1.27 1.27)) (justify left))
-    )
-  )
-  (sheet (at 171.45 63.5) (size 19.05 15.24) (fields_autoplaced)
-    (stroke (width 0.1524) (type solid) (color 0 0 0 0))
-    (fill (color 0 0 0 0.0000))
-    (property "Sheet name" "Current Sense A" (id 0) (at 171.45 62.7884 0)
-      (effects (font (size 1.27 1.27)) (justify left bottom))
-    )
-    (property "Sheet file" "CurrentSense.kicad_sch" (id 1) (at 171.45 79.3246 0)
-      (effects (font (size 1.27 1.27)) (justify left top))
-    )
-    (pin "GND" input (at 171.45 76.2 180)
-      (effects (font (size 1.27 1.27)) (justify left))
-    )
-    (pin "IS-" input (at 171.45 72.39 180)
-      (effects (font (size 1.27 1.27)) (justify left))
-    )
-    (pin "IS+" input (at 171.45 69.85 180)
-      (effects (font (size 1.27 1.27)) (justify left))
-    )
-    (pin "IOUT" input (at 190.5 68.58 0)
-      (effects (font (size 1.27 1.27)) (justify right))
-    )
-    (pin "VDD" input (at 171.45 66.04 180)
-      (effects (font (size 1.27 1.27)) (justify left))
-    )
-  )
-  (sheet (at 171.45 86.36) (size 19.05 15.24) (fields_autoplaced)
-    (stroke (width 0.1524) (type solid) (color 0 0 0 0))
-    (fill (color 0 0 0 0.0000))
-    (property "Sheet name" "Current Sense B" (id 0) (at 171.45 85.6484 0)
-      (effects (font (size 1.27 1.27)) (justify left bottom))
-    )
-    (property "Sheet file" "CurrentSense.kicad_sch" (id 1) (at 171.45 102.1846 0)
-      (effects (font (size 1.27 1.27)) (justify left top))
-    )
-    (pin "GND" input (at 171.45 99.06 180)
-      (effects (font (size 1.27 1.27)) (justify left))
-    )
-    (pin "IS-" input (at 171.45 95.25 180)
-      (effects (font (size 1.27 1.27)) (justify left))
-    )
-    (pin "IS+" input (at 171.45 92.71 180)
-      (effects (font (size 1.27 1.27)) (justify left))
-    )
-    (pin "IOUT" input (at 190.5 91.44 0)
-      (effects (font (size 1.27 1.27)) (justify right))
-    )
-    (pin "VDD" input (at 171.45 88.9 180)
+    (pin "VDD" input (at 186.69 88.9 180)
       (effects (font (size 1.27 1.27)) (justify left))
     )
@@
     )
   )
-  (sheet (at 86.36 63.5) (size 29.21 16.51) (fields_autoplaced)
-    (stroke (width 0.1524) (type solid) (color 0 0 0 0))
-    (fill (color 0 0 0 0.0000))
-    (property "Sheet name" "VGen" (id 0) (at 86.36 62.7884 0)
-      (effects (font (size 1.27 1.27)) (justify left bottom))
-    )
-    (property "Sheet file" "VGen.kicad_sch" (id 1) (at 86.36 80.5946 0)
-      (effects (font (size 1.27 1.27)) (justify left top))
-    )
-    (pin "3V3" input (at 115.57 68.58 0)
-      (effects (font (size 1.27 1.27)) (justify right))
-    )
-    (pin "12V0" input (at 115.57 66.04 0)
-      (effects (font (size 1.27 1.27)) (justify right))
-    )
-    (pin "GND" input (at 115.57 76.2 0)
-      (effects (font (size 1.27 1.27)) (justify right))
-    )
-    (pin "VIN" input (at 86.36 67.31 180)
-      (effects (font (size 1.27 1.27)) (justify left))
-    )
-  )

Commit message: Updated PCB
Other:
- sheet Current Sense Amp renamed Current Sense Amp A
- added sheet Current Sense Amp B (CurrentSense.kicad_sch)
- added sheet Current Sense Amp C (CurrentSense.kicad_sch)
Changed lines of the file:
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@@
     (stroke (width 0) (type default) (color 0 0 0 0))
+  )
+  (hierarchical_label "VDD" (shape input) (at 177.8 90.17 180)
+    (effects (font (size 1.27 1.27)) (justify right))
   )
   (hierarchical_label "V_{DRIVE}" (shape input) (at 115.57 66.04 180)
@@
     (effects (font (size 1.27 1.27)) (justify left))
   )
-  (hierarchical_label "I_{SENSE}" (shape input) (at 205.74 91.44 0)
+  (hierarchical_label "ISC" (shape input) (at 177.8 115.57 180)
+    (effects (font (size 1.27 1.27)) (justify right))
+  )
+  (hierarchical_label "I_{SENSE}A" (shape input) (at 196.85 68.58 0)
     (effects (font (size 1.27 1.27)) (justify left))
   )
@@
     (effects (font (size 1.27 1.27)) (justify left))
   )
-  (hierarchical_label "IS" (shape input) (at 186.69 92.71 180)
+  (hierarchical_label "I_{SENSE}B" (shape input) (at 196.85 92.71 0)
+    (effects (font (size 1.27 1.27)) (justify left))
+  )
+  (hierarchical_label "ISA" (shape input) (at 177.8 69.85 180)
     (effects (font (size 1.27 1.27)) (justify right))
   )
@@
     (effects (font (size 1.27 1.27)) (justify right))
   )
+  (hierarchical_label "I_{SENSE}C" (shape input) (at 196.85 114.3 0)
+    (effects (font (size 1.27 1.27)) (justify left))
+  )
   (hierarchical_label "CL" (shape input) (at 134.62 118.11 180)
     (effects (font (size 1.27 1.27)) (justify right))
   )
-  (hierarchical_label "GND" (shape input) (at 186.69 95.25 180)
+  (hierarchical_label "GND" (shape input) (at 177.8 72.39 180)
     (effects (font (size 1.27 1.27)) (justify right))
   )
@@
     (effects (font (size 1.27 1.27)) (justify right))
   )
+  (hierarchical_label "GND" (shape input) (at 177.8 121.92 180)
+    (effects (font (size 1.27 1.27)) (justify right))
+  )
   (hierarchical_label "C" (shape input) (at 158.75 116.84 0)
     (effects (font (size 1.27 1.27)) (justify left))
@@
   (hierarchical_label "GBH" (shape input) (at 158.75 91.44 0)
     (effects (font (size 1.27 1.27)) (justify left))
+  )
+  (hierarchical_label "GND" (shape input) (at 177.8 100.33 180)
+    (effects (font (size 1.27 1.27)) (justify right))
+  )
+  (hierarchical_label "GND" (shape input) (at 177.8 96.52 180)
+    (effects (font (size 1.27 1.27)) (justify right))
   )
   (hierarchical_label "GND" (shape input) (at 134.62 121.92 180)
@@
     (effects (font (size 1.27 1.27)) (justify left))
   )
-  (hierarchical_label "GND" (shape input) (at 186.69 99.06 180)
+  (hierarchical_label "GND" (shape input) (at 177.8 76.2 180)
+    (effects (font (size 1.27 1.27)) (justify right))
+  )
+  (hierarchical_label "VDD" (shape input) (at 177.8 111.76 180)
     (effects (font (size 1.27 1.27)) (justify right))
   )
@@
     (effects (font (size 1.27 1.27)) (justify right))
   )
-  (hierarchical_label "VDD" (shape input) (at 186.69 88.9 180)
+  (hierarchical_label "VDD" (shape input) (at 177.8 66.04 180)
+    (effects (font (size 1.27 1.27)) (justify right))
+  )
+  (hierarchical_label "GND" (shape input) (at 177.8 118.11 180)
     (effects (font (size 1.27 1.27)) (justify right))
   )
@@
     (effects (font (size 1.27 1.27)) (justify right))
   )
-  (sheet (at 186.69 86.36) (size 19.05 15.24) (fields_autoplaced)
+  (hierarchical_label "ISB" (shape input) (at 177.8 93.98 180)
+    (effects (font (size 1.27 1.27)) (justify right))
+  )
+  (sheet (at 177.8 63.5) (size 19.05 15.24) (fields_autoplaced)
     (stroke (width 0.1524) (type solid) (color 0 0 0 0))
     (fill (color 0 0 0 0.0000))
-    (property "Sheet name" "Current Sense Amp" (id 0) (at 186.69 85.6484 0)
+    (property "Sheet name" "Current Sense Amp A" (id 0) (at 177.8 62.7884 0)
       (effects (font (size 1.27 1.27)) (justify left bottom))
     )
-    (property "Sheet file" "CurrentSense.kicad_sch" (id 1) (at 186.69 102.1846 0)
+    (property "Sheet file" "CurrentSense.kicad_sch" (id 1) (at 177.8 79.3246 0)
       (effects (font (size 1.27 1.27)) (justify left top))
     )
-    (pin "GND" input (at 186.69 99.06 180)
+    (pin "GND" input (at 177.8 76.2 180)
       (effects (font (size 1.27 1.27)) (justify left))
     )
-    (pin "IS-" input (at 186.69 95.25 180)
+    (pin "IS-" input (at 177.8 72.39 180)
       (effects (font (size 1.27 1.27)) (justify left))
     )
-    (pin "IS+" input (at 186.69 92.71 180)
+    (pin "IS+" input (at 177.8 69.85 180)
       (effects (font (size 1.27 1.27)) (justify left))
     )
-    (pin "IOUT" input (at 205.74 91.44 0)
+    (pin "IOUT" input (at 196.85 68.58 0)
       (effects (font (size 1.27 1.27)) (justify right))
     )
-    (pin "VDD" input (at 186.69 88.9 180)
+    (pin "VDD" input (at 177.8 66.04 180)
       (effects (font (size 1.27 1.27)) (justify left))
     )
+  )
+  (sheet (at 177.8 109.22) (size 19.05 15.24) (fields_autoplaced)
+    (stroke (width 0.1524) (type solid) (color 0 0 0 0))
+    (fill (color 0 0 0 0.0000))
+    (property "Sheet name" "Current Sense Amp C" (id 0) (at 177.8 108.5084 0)
+      (effects (font (size 1.27 1.27)) (justify left bottom))
+    )
+    (property "Sheet file" "CurrentSense.kicad_sch" (id 1) (at 177.8 125.0446 0)
+      (effects (font (size 1.27 1.27)) (justify left top))
+    )
+    (pin "GND" input (at 177.8 121.92 180)
+      (effects (font (size 1.27 1.27)) (justify left))
+    )
+    (pin "IS-" input (at 177.8 118.11 180)
+      (effects (font (size 1.27 1.27)) (justify left))
+    )
+    (pin "IS+" input (at 177.8 115.57 180)
+      (effects (font (size 1.27 1.27)) (justify left))
+    )
+    (pin "IOUT" input (at 196.85 114.3 0)
+      (effects (font (size 1.27 1.27)) (justify right))
+    )
+    (pin "VDD" input (at 177.8 111.76 180)
+      (effects (font (size 1.27 1.27)) (justify left))
+    )
+  )
+  (sheet (at 177.8 87.63) (size 19.05 15.24) (fields_autoplaced)
+    (stroke (width 0.1524) (type solid) (color 0 0 0 0))
+    (fill (color 0 0 0 0.0000))
+    (property "Sheet name" "Current Sense Amp B" (id 0) (at 177.8 86.9184 0)
+      (effects (font (size 1.27 1.27)) (justify left bottom))
+    )
+    (property "Sheet file" "CurrentSense.kicad_sch" (id 1) (at 177.8 103.4546 0)
+      (effects (font (size 1.27 1.27)) (justify left top))
+    )
+    (pin "GND" input (at 177.8 100.33 180)
+      (effects (font (size 1.27 1.27)) (justify left))
+    )
+    (pin "IS-" input (at 177.8 96.52 180)
+      (effects (font (size 1.27 1.27)) (justify left))
+    )
+    (pin "IS+" input (at 177.8 93.98 180)
+      (effects (font (size 1.27 1.27)) (justify left))
+    )
+    (pin "IOUT" input (at 196.85 92.71 0)
+      (effects (font (size 1.27 1.27)) (justify right))
+    )
+    (pin "VDD" input (at 177.8 90.17 180)
+      (effects (font (size 1.27 1.27)) (justify left))
+    )
