File: OpenMC/Hi-LowDriver.kicad_sch (KiCad schematic)
At the start: 6 parts, among them U3 LT2190NTR

Commit message: pcb work
Parts:
- removed R11: R_US, Resistor_SMD:R_1206_3216Metric, symbol Device:R_US
- C2: renamed from C3; value C_Small -> 1uF; footprint (none) -> Resistor_SMD:R_0603_1608Metric
- R7: renamed from R10; value R_US -> 10
- R9: renamed from R12; value R_US -> 10
- renumbered D3 to D2, U3 to U2
Connections:
- net VDD: now also D2.2 (A)
Changed lines of the file:
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@@
     (stroke (width 0) (type default) (color 0 0 0 0))
   )
-  (hierarchical_label "VDD" (shape input) (at 161.29 80.01 90)
+  (hierarchical_label "VDD" (shape input) (at 161.29 87.63 90)
     (effects (font (size 1.27 1.27)) (justify left))
   )
@@
   (symbol (lib_id "OpenMC:LT2190NTR") (at 149.86 99.06 0)
     (in_bom yes) (on_board yes) (fields_autoplaced)
-    (property "Reference" "U3" (id 0) (at 149.86 88.7943 0))
+    (property "Reference" "U2" (id 0) (at 149.86 88.7943 0))
     (property "Value" "LT2190NTR" (id 1) (at 149.86 91.5694 0))
     (property "Footprint" "Package_SO:SOIC-8_3.9x4.9mm_P1.27mm" (id 2) (at 147.32 99.06 0)
@@
     (pin "8")
   )
-  (symbol (lib_id "Device:R_US") (at 161.29 83.82 0)
-    (in_bom yes) (on_board yes)
-    (property "Reference" "R11" (id 0) (at 158.75 85.09 90))
-    (property "Value" "R_US" (id 1) (at 163.3704 83.82 90)
-      (effects (font (size 1.27 1.27)) hide)
-    )
-    (property "Footprint" "Resistor_SMD:R_1206_3216Metric" (id 2) (at 162.306 84.074 90)
-      (effects (font (size 1.27 1.27)) hide)
-    )
-    (property "Datasheet" "~" (id 3) (at 161.29 83.82 0)
-      (effects (font (size 1.27 1.27)) hide)
-    )
-    (pin "1")
-    (pin "2")
-  )
   (symbol (lib_id "Device:R_US") (at 137.16 102.87 90)
     (in_bom yes) (on_board yes)
-    (property "Reference" "R10" (id 0) (at 137.16 105.41 90))
-    (property "Value" "R_US" (id 1) (at 137.16 100.7896 90)
+    (property "Reference" "R7" (id 0) (at 137.16 105.41 90))
+    (property "Value" "10" (id 1) (at 137.16 100.7896 90)
       (effects (font (size 1.27 1.27)) hide)
     )
@@
   (symbol (lib_id "Device:C_Small") (at 173.99 97.79 0)
     (in_bom yes) (on_board yes)
-    (property "Reference" "C3" (id 0) (at 176.3141 96.8878 0)
+    (property "Reference" "C2" (id 0) (at 176.3141 96.8878 0)
       (effects (font (size 1.27 1.27)) (justify left))
     )
-    (property "Value" "C_Small" (id 1) (at 176.53 99.06 0)
-      (effects (font (size 1.27 1.27)) (justify left) hide)
+    (property "Value" "1uF" (id 1) (at 176.53 99.06 0)
+      (effects (font (size 1.27 1.27)) (justify left))
     )
-    (property "Footprint" "" (id 2) (at 173.99 97.79 0)
+    (property "Footprint" "Resistor_SMD:R_0603_1608Metric" (id 2) (at 173.99 97.79 0)
       (effects (font (size 1.27 1.27)) hide)
     )
@@
   (symbol (lib_id "Device:D") (at 161.29 91.44 90)
     (in_bom yes) (on_board yes) (fields_autoplaced)
-    (property "Reference" "D3" (id 0) (at 163.322 90.5315 90)
+    (property "Reference" "D2" (id 0) (at 163.322 90.5315 90)
       (effects (font (size 1.27 1.27)) (justify right))
     )
@@
   (symbol (lib_id "Device:R_US") (at 162.56 97.79 90)
     (in_bom yes) (on_board yes)
-    (property "Reference" "R12" (id 0) (at 165.1 96.52 90))
-    (property "Value" "R_US" (id 1) (at 162.56 95.7096 90)
+    (property "Reference" "R9" (id 0) (at 165.1 96.52 90))
+    (property "Value" "10" (id 1) (at 162.56 95.7096 90)
       (effects (font (size 1.27 1.27)) hide)
     )

Commit message: Updated PCB
Parts:
- added C5: 1uF, Resistor_SMD:R_0603_1608Metric, symbol Device:C_Small
- renumbered C2 to C1, D2 to D1, R7 to R4, R9 to R6, U2 to U1
Connections:
- net GND: now also C5.2
- net VDD: now also C5.1
Changed lines of the file:
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@@
 (kicad_sch (version 20211123) (generator eeschema)
   (paper "A4")
+  (junction (at 161.29 102.87) (diameter 0) (color 0 0 0 0)
+  )
   (junction (at 161.29 95.25) (diameter 0) (color 0 0 0 0)
   )
   (junction (at 173.99 100.33) (diameter 0) (color 0 0 0 0)
+  )
+  (wire (pts (xy 166.37 102.87) (xy 161.29 102.87))
+    (stroke (width 0) (type default) (color 0 0 0 0))
   )
   (wire (pts (xy 161.29 95.25) (xy 158.75 95.25))
@@
   )
   (wire (pts (xy 175.26 100.33) (xy 173.99 100.33))
+    (stroke (width 0) (type default) (color 0 0 0 0))
+  )
+  (wire (pts (xy 161.29 102.87) (xy 158.75 102.87))
     (stroke (width 0) (type default) (color 0 0 0 0))
   )
@@
     (effects (font (size 1.27 1.27)) (justify right))
   )
-  (hierarchical_label "VDD" (shape input) (at 158.75 102.87 0)
+  (hierarchical_label "GND" (shape input) (at 161.29 107.95 270)
+    (effects (font (size 1.27 1.27)) (justify right))
+  )
+  (hierarchical_label "VDD" (shape input) (at 166.37 102.87 0)
     (effects (font (size 1.27 1.27)) (justify left))
   )
@@
   (symbol (lib_id "OpenMC:LT2190NTR") (at 149.86 99.06 0)
     (in_bom yes) (on_board yes) (fields_autoplaced)
-    (property "Reference" "U2" (id 0) (at 149.86 88.7943 0))
+    (property "Reference" "U1" (id 0) (at 149.86 88.7943 0))
     (property "Value" "LT2190NTR" (id 1) (at 149.86 91.5694 0))
     (property "Footprint" "Package_SO:SOIC-8_3.9x4.9mm_P1.27mm" (id 2) (at 147.32 99.06 0)
@@
     (pin "8")
   )
+  (symbol (lib_id "Device:C_Small") (at 161.29 105.41 0)
+    (in_bom yes) (on_board yes)
+    (property "Reference" "C5" (id 0) (at 163.6141 104.5078 0)
+      (effects (font (size 1.27 1.27)) (justify left))
+    )
+    (property "Value" "1uF" (id 1) (at 163.83 106.68 0)
+      (effects (font (size 1.27 1.27)) (justify left))
+    )
+    (property "Footprint" "Resistor_SMD:R_0603_1608Metric" (id 2) (at 161.29 105.41 0)
+      (effects (font (size 1.27 1.27)) hide)
+    )
+    (property "Datasheet" "~" (id 3) (at 161.29 105.41 0)
+      (effects (font (size 1.27 1.27)) hide)
+    )
+    (pin "1")
+    (pin "2")
+  )
   (symbol (lib_id "Device:R_US") (at 137.16 102.87 90)
     (in_bom yes) (on_board yes)
-    (property "Reference" "R7" (id 0) (at 137.16 105.41 90))
+    (property "Reference" "R4" (id 0) (at 137.16 105.41 90))
     (property "Value" "10" (id 1) (at 137.16 100.7896 90)
       (effects (font (size 1.27 1.27)) hide)
@@
   (symbol (lib_id "Device:C_Small") (at 173.99 97.79 0)
     (in_bom yes) (on_board yes)
-    (property "Reference" "C2" (id 0) (at 176.3141 96.8878 0)
+    (property "Reference" "C1" (id 0) (at 176.3141 96.8878 0)
       (effects (font (size 1.27 1.27)) (justify left))
     )
@@
   (symbol (lib_id "Device:D") (at 161.29 91.44 90)
     (in_bom yes) (on_board yes) (fields_autoplaced)
-    (property "Reference" "D2" (id 0) (at 163.322 90.5315 90)
+    (property "Reference" "D1" (id 0) (at 163.322 90.5315 90)
       (effects (font (size 1.27 1.27)) (justify right))
     )
@@
   (symbol (lib_id "Device:R_US") (at 162.56 97.79 90)
     (in_bom yes) (on_board yes)
-    (property "Reference" "R9" (id 0) (at 165.1 96.52 90))
+    (property "Reference" "R6" (id 0) (at 165.1 96.52 90))
     (property "Value" "10" (id 1) (at 162.56 95.7096 90)
       (effects (font (size 1.27 1.27)) hide)
