File: OpenMC/OpenMC.kicad_pcb (KiCad board)
At the start: 2 copper layers, 42 parts, among them IC1 EFM8LB11F32E-C-QFN24, J1 Conn_01x05_Female, J10 Conn_01x01_Female, J11 Conn_01x01_Female, J2 Conn_01x01_Female, J3 Conn_01x01_Female, J4 Conn_01x06_Female, J5 Conn_01x01_Female, J6 Conn_01x01_Female, J7 Conn_01x05_Female, J8 Conn_01x01_Female, J9 Conn_01x01_Female, Q1 BSC026N08NS5, Q10 BSC026N08NS5, Q11 BSC026N08NS5, Q12 BSC026N08NS5, Q13 BSC026N08NS5, Q14 BSC026N08NS5, Q15 BSC026N08NS5, Q16 BSC026N08NS5, Q17 BSC026N08NS5, Q18 BSC026N08NS5, Q19 BSC026N08NS5, Q2 BSC026N08NS5, Q20 BSC026N08NS5, Q21 BSC026N08NS5, Q22 BSC026N08NS5, Q23 BSC026N08NS5, Q24 BSC026N08NS5, Q3 BSC026N08NS5, Q4 BSC026N08NS5, Q5 BSC026N08NS5, Q6 BSC026N08NS5, Q7 BSC026N08NS5, Q8 BSC026N08NS5, Q9 BSC026N08NS5

Commit message: updates
Parts:
- removed J10, J11, J8, J9: Conn_01x01_Female, Connector:Banana_Jack_1Pin
- removed Q13, Q14, Q15, Q16, Q17, Q18, Q19, Q20, Q21, Q22, Q23, Q24: BSC026N08NS5, Package_TO_SOT_SMD:TDSON-8-1
- added C10: C, Capacitor_SMD:C_0603_1608Metric, B.Cu at (215.9, 111.9)
- added C11: C, Capacitor_SMD:C_0603_1608Metric, B.Cu at (125.6, 134.0)
- added C12: C, Capacitor_SMD:C_0603_1608Metric, B.Cu at (137.8, 133.9)
- added C13: C, Capacitor_SMD:C_0603_1608Metric, B.Cu at (150.2, 133.9)
- added C14: C, Capacitor_SMD:C_0603_1608Metric, B.Cu at (139.3, 133.9)
- added C15: C, Capacitor_SMD:C_0603_1608Metric, B.Cu at (127.1, 134.0)
- added C16: C, Capacitor_SMD:C_0603_1608Metric, B.Cu at (216.4, 120.4)
- added C20: C, Capacitor_SMD:C_1210_3225Metric, F.Cu at (165.5, 104.0)
- added C4: .1uF, Diode_SMD:D_0603_1608Metric, B.Cu at (208.2, 106.7)
- added C5: .1uF, Diode_SMD:D_0603_1608Metric, B.Cu at (218.9, 108.1)
- added C6: C, Capacitor_SMD:C_1210_3225Metric, F.Cu at (155.8, 104.0)
- added C7: C, Capacitor_SMD:C_1210_3225Metric, F.Cu at (159.0, 104.0)
- added C8: C, Capacitor_SMD:C_1210_3225Metric, F.Cu at (162.3, 104.0)
- added C9: C, Capacitor_SMD:C_0603_1608Metric, B.Cu at (119.8, 134.0)
- added D1: D, Diode_SMD:D_1206_3216Metric, B.Cu at (133.9, 123.7)
- added D2: D, Diode_SMD:D_1206_3216Metric, B.Cu at (146.4, 123.7)
- added D3: D, Diode_SMD:D_1206_3216Metric, B.Cu at (121.7, 123.7)
- added IC2: BD9G341AEFJ-E2, SamacSys_Parts:SOIC127P600X100-9N, B.Cu at (213.5, 107.3)
- added IC3: XC9236A18CMR-G, SamacSys_Parts:SOT95P280X130-5N, B.Cu at (215.6, 114.9)
- added IC4: INA186A4QDBVRQ1, SamacSys_Parts:SOT95P280X145-5N, B.Cu at (154.1, 130.0)
- added IC5: INA186A4QDBVRQ1, SamacSys_Parts:SOT95P280X145-5N, B.Cu at (142.2, 130.0)
- added IC6: INA186A4QDBVRQ1, SamacSys_Parts:SOT95P280X145-5N, B.Cu at (129.7, 130.0)
- added L1: 33uH, Inductor_SMD:L_Taiyo-Yuden_NR-60xx, B.Cu at (210.1, 113.8)
- added L2: L, Inductor_SMD:L_1206_3216Metric, B.Cu at (215.6, 118.4)
- added R10: R_US, Resistor_SMD:R_1206_3216Metric, B.Cu at (128.1, 124.8)
- added R11: R_US, Resistor_SMD:R_1206_3216Metric, B.Cu at (118.1, 124.8)
- added R12: R_US, Resistor_SMD:R_1206_3216Metric, B.Cu at (125.9, 124.8)
- added R13: R_US, Resistor_SMD:R_0603_1608Metric, B.Cu at (208.2, 103.6)
- added R14: R_US, Resistor_SMD:R_0603_1608Metric, B.Cu at (208.2, 105.2)
- added R15: R_US, Resistor_SMD:R_0603_1608Metric, B.Cu at (208.2, 108.2)
- added R16: R_US, Resistor_SMD:R_0603_1608Metric, B.Cu at (218.9, 109.6)
- added R17: R_US, Resistor_SMD:R_0603_1608Metric, B.Cu at (218.9, 106.6)
- added R18: R_US, Capacitor_SMD:C_0603_1608Metric, B.Cu at (148.7, 133.9)
- added R19: R_US, Resistor_SMD:R_0603_1608Metric, B.Cu at (218.9, 105.0)
- added R20: R_US, Capacitor_SMD:C_0603_1608Metric, B.Cu at (136.3, 133.9)
- added R21: R_US, Capacitor_SMD:C_0603_1608Metric, B.Cu at (124.1, 134.0)
- added R22: R_US, Capacitor_SMD:C_0603_1608Metric, B.Cu at (147.2, 133.9)
- added R23: R_US, Capacitor_SMD:C_0603_1608Metric, B.Cu at (134.7, 133.9)
- added R24: R_US, Capacitor_SMD:C_0603_1608Metric, B.Cu at (122.6, 134.0)
- added R7: R_US, Resistor_SMD:R_1206_3216Metric, B.Cu at (152.9, 124.8)
- added R8: R_US, Resistor_SMD:R_1206_3216Metric, B.Cu at (142.6, 124.8)
- added R9: R_US, Resistor_SMD:R_1206_3216Metric, B.Cu at (150.6, 124.8)
- added U1: LT2190NTR, Package_SO:SOIC-8_3.9x4.9mm_P1.27mm, B.Cu at (134.2, 128.5)
- added U2: LT2190NTR, Package_SO:SOIC-8_3.9x4.9mm_P1.27mm, B.Cu at (146.8, 128.5)
- added U3: LT2190NTR, Package_SO:SOIC-8_3.9x4.9mm_P1.27mm, B.Cu at (122.0, 128.7)
- IC1: value EFM8LB11F32E-C-QFN24 -> EFM8BB31F32G-D-QSOP24R; footprint SamacSys_Parts:EFM8LB11F32EBQFN24R -> SamacSys_Parts:SOP64P600X175-24N; moved to B.Cu
- J1: value Conn_01x05_Female -> Conn_01x01_Female; footprint Connector_PinSocket_2.54mm:PinSocket_1x05_P2.54mm_Vertical -> Connector:Banana_Jack_1Pin
- J3: value Conn_01x01_Female -> Power+
- J4: value Conn_01x06_Female -> Control
- J5: value Conn_01x01_Female -> Power-
- J7: value Conn_01x05_Female -> Hall Connector; footprint Connector_PinSocket_2.54mm:PinSocket_1x05_P2.54mm_Vertical -> Connector_PinHeader_2.00mm:PinHeader_1x05_P2.00mm_Vertical
- R4, R5, R6: value WSL36371L000DEA -> R_US; footprint SamacSys_Parts:WSL36371L000DEA -> Resistor_SMD:R_1206_3216Metric; moved to B.Cu
- moved J4 113.3 mm to (136.9, 145.8), turned to 90 degrees
- moved J7 109.3 mm to (117.2, 137.7)
- moved IC1 104.2 mm to (137.0, 140.1), turned to 90 degrees
- moved J5 68.5 mm to (160.9, 140.3)
- moved J1 67.1 mm to (146.8, 111.1)
- moved R6 63.7 mm to (138.0, 124.8), turned to 90 degrees
- moved J3 63.5 mm to (160.7, 96.5)
- moved J2 45.3 mm to (134.6, 111.1)
- moved J6 45.3 mm to (122.6, 111.1)
- moved Q6 35.2 mm to (137.5, 120.7)
- moved Q8 35.2 mm to (131.8, 120.7)
- moved Q12 35.2 mm to (125.6, 120.7)
- moved Q10 35.2 mm to (119.9, 120.7)
- moved Q2 35.2 mm to (149.7, 120.7)
- moved Q4 35.2 mm to (144.0, 120.7)
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Connections:
- net /Left Hall Sensors/HA renamed /Controller/HALL_A
- net /Left Hall Sensors/HB renamed /Controller/HALL_B
- net /Left Hall Sensors/HC renamed /Controller/HALL_C
- net /Right Driver FETs/AH renamed /Driver FETs/AH
- net /Right Driver FETs/AL renamed /Driver FETs/AL
- net /Right Driver FETs/CH renamed /Driver FETs/CH
- net /Right Driver FETs/CL renamed /Driver FETs/CL
- net /Right Driver FETs/ISA renamed /Driver FETs/ISA
- net /Right Driver FETs/ISB renamed /Driver FETs/ISB
- net /Right Driver FETs/ISC renamed /Driver FETs/ISC
- IC1 pad 1: unconnected-(IC1-Pad1) -> /Controller/MOSI
- IC1 pad 10: /BRAKE -> unconnected-(IC1-Pad10)
- IC1 pad 11: /PWM -> unconnected-(IC1-Pad11)
- IC1 pad 13: unconnected-(IC1-Pad13) -> /Controller/ISC
- IC1 pad 14: unconnected-(IC1-Pad14) -> /Controller/ISB
- IC1 pad 15: /GND -> /Controller/ISA
- IC1 pad 19: unconnected-(IC1-Pad19) -> /Controller/CH
- IC1 pad 2: unconnected-(IC1-Pad2) -> /Controller/MISO
- IC1 pad 20: unconnected-(IC1-Pad20) -> /Controller/CL
- IC1 pad 21: unconnected-(IC1-Pad21) -> /Controller/BL
- IC1 pad 22: unconnected-(IC1-Pad22) -> /Controller/BH
- IC1 pad 23: unconnected-(IC1-Pad23) -> /Controller/AL
- IC1 pad 24: unconnected-(IC1-Pad24) -> /Controller/AH
- IC1 pad 3: /GND -> /Controller/SCLK
- IC1 pad 4: /VDD -> /Controller/CS
- IC1 pad 5: /RST -> /Controller/GND
- IC1 pad 6: unconnected-(IC1-Pad6) -> /VDD
- IC1 pad 7: unconnected-(IC1-Pad7) -> /C2CK
- IC1 pad 8: /EN -> /C2D
- IC1 pad 9: /COAST -> unconnected-(IC1-Pad9)
- J1 pad 1: /Right Hall Sensors/GND -> /A
- J2 pad 1: /Right Driver FETs/A -> /B
- J4 pad 1: /GND -> /Controller/GND
- J4 pad 2: /EN -> /Controller/CS
- J4 pad 3: /COAST -> /Controller/SCLK
- J4 pad 4: /BRAKE -> /Controller/MISO
- J4 pad 5: /PWM -> /Controller/MOSI
- J6 pad 1: /Right Driver FETs/B -> /C
- J7 pad 1: /Left Hall Sensors/GND -> Earth
- J7 pad 5: /Left Hall Sensors/VDD -> /VDD
- Q1 pad 1: /Right Driver FETs/A -> /A
- Q1 pad 2: /Right Driver FETs/A -> /A
- Q1 pad 3: /Right Driver FETs/A -> /A
- Q10 pad 5: /Right Driver FETs/C -> /C
- Q11 pad 1: /Right Driver FETs/C -> /C
- Q11 pad 2: /Right Driver FETs/C -> /C
- Q11 pad 3: /Right Driver FETs/C -> /C
- Q12 pad 5: /Right Driver FETs/C -> /C
- Q2 pad 5: /Right Driver FETs/A -> /A
- Q3 pad 1: /Right Driver FETs/A -> /A
- Q3 pad 2: /Right Driver FETs/A -> /A
- Q3 pad 3: /Right Driver FETs/A -> /A
- Q4 pad 5: /Right Driver FETs/A -> /A
- Q5 pad 1: /Right Driver FETs/B -> /B
- Q5 pad 2: /Right Driver FETs/B -> /B
- Q5 pad 3: /Right Driver FETs/B -> /B
- Q5 pad 4: /Right Driver FETs/BH -> /Driver FETs/BH
- Q6 pad 4: /Right Driver FETs/BL -> /Driver FETs/BL
- Q6 pad 5: /Right Driver FETs/B -> /B
- Q7 pad 1: /Right Driver FETs/B -> /B
- Q7 pad 2: /Right Driver FETs/B -> /B
- Q7 pad 3: /Right Driver FETs/B -> /B
- Q7 pad 4: /Right Driver FETs/BH -> /Driver FETs/BH
- Q8 pad 4: /Right Driver FETs/BL -> /Driver FETs/BL
- Q8 pad 5: /Right Driver FETs/B -> /B
- Q9 pad 1: /Right Driver FETs/C -> /C
- Q9 pad 2: /Right Driver FETs/C -> /C
- Q9 pad 3: /Right Driver FETs/C -> /C
- R1 pad E1: /Right Driver FETs/ISA+ -> /Driver FETs/ISA+
- R1 pad E2: /Right Driver FETs/ISA- -> Earth
- R2 pad E1: /Right Driver FETs/ISB+ -> /Driver FETs/ISB+
- R2 pad E2: /Right Driver FETs/ISB- -> Earth
- R3 pad E1: /Right Driver FETs/ISC+ -> /Driver FETs/ISC+
- R3 pad E2: /Right Driver FETs/ISC- -> Earth
Routing:
- net /Pre-Driver/A Driver/VDD: track 0.00 -> 63.5 mm, vias 0 -> 1
- net /Driver FETs/BH: track 0.00 -> 34.3 mm, vias 0 -> 1
- net Net-(IC2-Pad1): track 0.00 -> 33.9 mm
- net /Driver FETs/CH: track 0.00 -> 31.1 mm, vias 0 -> 1
- net /Driver FETs/AH: track 6.96 -> 30.6 mm, vias 0 -> 1
- net /Pre-Driver/3V3: track 0.00 -> 15.9 mm
- net +BATT: track 0.00 -> 15.2 mm, vias 0 -> 150
- net Net-(R7-Pad2): track 0.00 -> 11.1 mm
- net /Driver FETs/AL: track 0.72 -> 11.7 mm, vias 0 -> 1
- net Net-(R4-Pad2): track 0.00 -> 11.0 mm
- net Net-(R10-Pad2): track 0.00 -> 10.9 mm
- net /Driver FETs/BL: track 0.00 -> 9.87 mm, vias 0 -> 1
- net /Driver FETs/CL: track 0.00 -> 9.82 mm, vias 0 -> 1
- net /Right Driver FETs/BH: track 6.96 -> 0.00 mm
- net Net-(R9-Pad1): track 0.00 -> 6.48 mm
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- added copper zone on B.Cu, net +BATT
- added copper zone on B.Cu, net /A
- added copper zone on F.Cu, net /A
- added copper zone on B.Cu, net /B
- added copper zone on F.Cu, net /B
- added copper zone on B.Cu, net /C
- added copper zone on F.Cu, net /C
- added copper zone on B.Cu, net Earth
- removed copper zone on F.Cu, net /Left Driver FETs/A
- removed copper zone on F.Cu, net /Left Driver FETs/B
- removed copper zone on F.Cu, net /Right Driver FETs/A
- removed copper zone on F.Cu, net /Right Driver FETs/B
- removed copper zone on F.Cu, net /Right Driver FETs/C
Other:
- board outline added: 53.3 x 57.8 mm

Commit message: pcb work
Parts:
- removed C14, C15, C16: C, Capacitor_SMD:C_0603_1608Metric
- removed C20: C, Capacitor_SMD:C_1210_3225Metric
- removed the C5 at (218.9, 108.1)
- removed IC2: BD9G341AEFJ-E2, SamacSys_Parts:SOIC127P600X100-9N
- removed IC3: XC9236A18CMR-G, SamacSys_Parts:SOT95P280X130-5N
- removed IC5, IC6: INA186A4QDBVRQ1, SamacSys_Parts:SOT95P280X145-5N
- removed L1: 33uH, Inductor_SMD:L_Taiyo-Yuden_NR-60xx
- removed L2: L, Inductor_SMD:L_1206_3216Metric
- removed R11, R5, R8: R_US, Resistor_SMD:R_1206_3216Metric
- removed R15, R16, R17, R19: R_US, Resistor_SMD:R_0603_1608Metric
- removed R18, R20, R21, R22, R23, R24: R_US, Capacitor_SMD:C_0603_1608Metric
- added C1: 1uF, Resistor_SMD:R_0603_1608Metric, B.Cu at (135.0, 121.8)
- added C2: 1uF, Resistor_SMD:R_0603_1608Metric, B.Cu at (147.6, 122.1)
- added C3: 1uF, Resistor_SMD:R_0603_1608Metric, B.Cu at (122.8, 122.1)
- added C5: .1uF, Capacitor_SMD:C_0603_1608Metric, F.Cu at (177.8, 120.0)
- added C5: 27uF, Capacitor_THT:C_Radial_D6.3mm_H7.0mm_P2.50mm, B.Cu at (160.3, 130.2)
- added J8: 216990-0001, SamacSys_Parts:2169900001, B.Cu at (189.2, 109.1)
- added Q13: 2N7002E, Package_TO_SOT_SMD:SOT-23, B.Cu at (231.1, 115.8)
- added Q14: VP0610T, Package_TO_SOT_SMD:SOT-23, B.Cu at (227.1, 115.8)
- added Q15: 2N7002E, Package_TO_SOT_SMD:SOT-23, B.Cu at (227.1, 119.2)
- added Q16: VP0610T, Package_TO_SOT_SMD:SOT-23, B.Cu at (231.1, 119.2)
- added U4: LM3480-3.3, Package_TO_SOT_SMD:SOT-23, B.Cu at (195.4, 150.0)
- added Y1: 40MHz, SamacSys_Parts:ABM12W300000MHZ6B1UT3, B.Cu at (223.6, 150.4)
- C10, C11, C12, C13, C9: value C -> 1uF
- C4: value .1uF -> 27uF; footprint Diode_SMD:D_0603_1608Metric -> Capacitor_THT:C_Radial_D6.3mm_H7.0mm_P2.50mm
- C6, C7, C8: value C -> 27uF; footprint Capacitor_SMD:C_1210_3225Metric -> Capacitor_THT:C_Radial_D6.3mm_H7.0mm_P2.50mm; moved to B.Cu
- IC1: value EFM8BB31F32G-D-QSOP24R -> ESP32-C3; footprint SamacSys_Parts:SOP64P600X175-24N -> SamacSys_Parts:QFN50P500X500X90-33N-D
- J7: footprint Connector_PinHeader_2.00mm:PinHeader_1x05_P2.00mm_Vertical -> Connector_JST:JST_PH_B5B-PH-K_1x05_P2.00mm_Vertical; moved to B.Cu
- Q1, Q10, Q11, Q12, Q2, Q3, Q4, Q5, Q6, Q7, Q8, Q9: value BSC026N08NS5 -> SIR188DP; footprint Package_TO_SOT_SMD:TDSON-8-1 -> Package_SO:PowerPAK_SO-8_Single
- R1, R2, R3: value WSL36371L000DEA -> PSR400ITQFL3L00; footprint SamacSys_Parts:WSL36371L000DEA -> SamacSys_Parts:RESC10052X200N
- R13, R14: value R_US -> 10k
- moved R13 92.9 mm to (135.0, 160.8)
- moved C9 88.9 mm to (208.6, 133.1), turned to 180 degrees
- moved C11 86.2 mm to (207.1, 162.1), turned to 180 degrees
- moved J4 84.7 mm to (221.2, 136.9), turned to -90 degrees
- moved C12 83.9 mm to (221.0, 123.1), turned to 90 degrees
- moved J7 77.7 mm to (194.9, 137.0), turned to 90 degrees
- moved C10 77.4 mm to (153.7, 158.0), turned to 90 degrees
- moved C13 68.1 mm to (211.1, 164.6), turned to 180 degrees
- moved C4 48.0 mm to (160.3, 108.8)
- moved R14 45.6 mm to (209.6, 150.8), turned to 180 degrees
- moved IC1 40.8 mm to (175.8, 152.8), turned to 180 degrees
- moved C6 19.6 mm to (160.3, 123.1), turned to 180 degrees
- moved R2 12.5 mm to (147.0, 128.4), turned to 90 degrees
- moved R1 12.2 mm to (134.8, 128.4), turned to 90 degrees
- moved C7 12.0 mm to (160.3, 116.0), turned to 180 degrees
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Connections:
- net /C2CK renamed /Controller/RST
- C10 pad 1: /Pre-Driver/A Driver/VDD -> /Controller/VDD
- C11 pad 1: /Pre-Driver/A Driver/VDD -> /Controller/VDD
- C12 pad 1: /Pre-Driver/A Driver/VDD -> /Controller/VDD
- C13 pad 1: /Pre-Driver/3V3 -> /Controller/VDD
- C4 pad 1: Net-(IC2-Pad3) -> +BATT
- C4 pad 2: Net-(C4-Pad2) -> Earth
- C9 pad 1: /Pre-Driver/A Driver/VDD -> /Controller/VBUS
- D1 pad 2: Net-(D1-Pad2) -> /Pre-Driver/V_{DRIVE}
- D2 pad 2: Net-(D2-Pad2) -> /Pre-Driver/V_{DRIVE}
- D3 pad 2: Net-(D3-Pad2) -> /Pre-Driver/V_{DRIVE}
- IC1 pad 1: /Controller/MOSI -> unconnected-(IC1-Pad1)
- IC1 pad 11: unconnected-(IC1-Pad11) -> /Controller/VDD
- IC1 pad 12: unconnected-(IC1-Pad12) -> /Controller/BL
- IC1 pad 13: /Controller/ISC -> /Controller/BH
- IC1 pad 14: /Controller/ISB -> /Controller/AL
- IC1 pad 15: /Controller/ISA -> /Controller/AH
- IC1 pad 17: unconnected-(IC1-Pad17) -> /Controller/VDD
- IC1 pad 18: unconnected-(IC1-Pad18) -> /Controller/VDD
- IC1 pad 19: /Controller/CH -> unconnected-(IC1-Pad19)
- IC1 pad 2: /Controller/MISO -> /Controller/VDD
- IC1 pad 20: /Controller/CL -> unconnected-(IC1-Pad20)
- IC1 pad 21: /Controller/BL -> /Controller/CS
- IC1 pad 22: /Controller/BH -> /Controller/SCLK
- IC1 pad 23: /Controller/AL -> /Controller/MOSI
- IC1 pad 24: /Controller/AH -> /Controller/MISO
- IC1 pad 3: /Controller/SCLK -> /Controller/VDD
- IC1 pad 4: /Controller/CS -> /Controller/HALL_A
- IC1 pad 5: /Controller/GND -> /Controller/HALL_B
- IC1 pad 6: /VDD -> /Controller/HALL_C
- IC1 pad 8: /C2D -> /Controller/I_{SENSE}
- IC1 pad 9: unconnected-(IC1-Pad9) -> /Controller/V_{TEMP}
- IC4 pad 2: /Controller/ISA -> /Controller/I_{SENSE}
- IC4 pad 3: /Pre-Driver/3V3 -> /VDD
- IC4 pad 4: /Driver FETs/ISA+ -> /Driver FETs/IS
- J4 pad 1: /Controller/GND -> Earth
- Q10 pad 1: /Driver FETs/ISC -> /Driver FETs/IS
- Q10 pad 2: /Driver FETs/ISC -> /Driver FETs/IS
- Q10 pad 3: /Driver FETs/ISC -> /Driver FETs/IS
- Q12 pad 1: /Driver FETs/ISC -> /Driver FETs/IS
- Q12 pad 2: /Driver FETs/ISC -> /Driver FETs/IS
- Q12 pad 3: /Driver FETs/ISC -> /Driver FETs/IS
- Q2 pad 1: /Driver FETs/ISA -> /Driver FETs/IS
- Q2 pad 2: /Driver FETs/ISA -> /Driver FETs/IS
- Q2 pad 3: /Driver FETs/ISA -> /Driver FETs/IS
- Q4 pad 1: /Driver FETs/ISA -> /Driver FETs/IS
- Q4 pad 2: /Driver FETs/ISA -> /Driver FETs/IS
- Q4 pad 3: /Driver FETs/ISA -> /Driver FETs/IS
- Q6 pad 1: /Driver FETs/ISB -> /Driver FETs/IS
- Q6 pad 2: /Driver FETs/ISB -> /Driver FETs/IS
- Q6 pad 3: /Driver FETs/ISB -> /Driver FETs/IS
- Q8 pad 1: /Driver FETs/ISB -> /Driver FETs/IS
- Q8 pad 2: /Driver FETs/ISB -> /Driver FETs/IS
- Q8 pad 3: /Driver FETs/ISB -> /Driver FETs/IS
- R13 pad 1: /Pre-Driver/VGen/FB -> /Controller/3V3USB
- R13 pad 2: /Pre-Driver/A Driver/VDD -> Net-(Q13-Pad3)
- R14 pad 1: Earth -> /Controller/3V3
- R14 pad 2: /Pre-Driver/VGen/FB -> Net-(Q15-Pad3)
- U1 pad 1: /Pre-Driver/BH -> /Controller/BH
- U1 pad 2: /Pre-Driver/BL -> /Controller/BL
- U1 pad 5: /Pre-Driver/A Driver/VDD -> /Pre-Driver/V_{DRIVE}
- U2 pad 1: /Pre-Driver/AH -> /Controller/AH
- U2 pad 2: /Pre-Driver/AL -> /Controller/AL
- U2 pad 5: /Pre-Driver/A Driver/VDD -> /Pre-Driver/V_{DRIVE}
- U3 pad 1: /Pre-Driver/CH -> /Controller/CH
- U3 pad 2: /Pre-Driver/CL -> /Controller/CL
- U3 pad 5: /Pre-Driver/A Driver/VDD -> /Pre-Driver/V_{DRIVE}
Routing:
- net /Pre-Driver/V_{DRIVE}: track 0.00 -> 67.7 mm, vias 0 -> 3
- net /Pre-Driver/A Driver/VDD: track 63.5 -> 0.00 mm, vias 1 -> 0
- net Net-(IC2-Pad1): track 33.9 -> 0.00 mm
- net /Pre-Driver/3V3: track 15.9 -> 0.00 mm
- net +BATT: track 15.2 -> 0.00 mm, vias 150 -> 120
- net /Driver FETs/IS: track 0.00 -> 11.9 mm, vias 0 -> 1
- net Net-(C1-Pad1): track 2.72 -> 12.1 mm
- net /Controller/D-: track 0.00 -> 7.99 mm
- net /Controller/VBUS: track 0.00 -> 7.75 mm
- net /Controller/HALL_A: track 0.00 -> 7.62 mm
- net /Controller/HALL_C: track 0.00 -> 7.34 mm
- net /Controller/D+: track 0.00 -> 7.33 mm
- net Net-(C3-Pad1): track 2.84 -> 9.84 mm
- net /Controller/HALL_B: track 0.00 -> 7.00 mm
- net Net-(C2-Pad1): track 2.72 -> 9.70 mm
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- added copper zone on F.Cu, net /Driver FETs/IS
- removed copper zone on F.Cu, net /Driver FETs/ISA
- removed copper zone on F.Cu, net /Driver FETs/ISB
- removed copper zone on F.Cu, net /Driver FETs/ISC
Other:
- board size 53.3 x 57.8 mm -> 50.8 x 63.5 mm

Commit message: Updated PCB
Parts:
- removed the C5 at (177.8, 120.0)
- removed the C5 at (160.3, 130.2)
- removed Q13, Q15: 2N7002E, Package_TO_SOT_SMD:SOT-23
- removed Q14, Q16: VP0610T, Package_TO_SOT_SMD:SOT-23
- added C14: 1uF, Resistor_SMD:R_0603_1608Metric, B.Cu at (145.0, 121.4)
- added C15: 1uF, Resistor_SMD:R_0603_1608Metric, B.Cu at (132.5, 121.4)
- added C5: 1uF, Resistor_SMD:R_0603_1608Metric, B.Cu at (120.3, 121.5)
- added IC2: INA186A4QDBVRQ1, SamacSys_Parts:SOT95P280X145-5N, B.Cu at (138.9, 128.1)
- added IC3: INA186A4QDBVRQ1, SamacSys_Parts:SOT95P280X145-5N, B.Cu at (126.7, 128.4)
- added J9: Gate Drive Voltage, Connector_PinHeader_2.54mm:PinHeader_1x01_P2.54mm_Vertical, F.Cu at (117.6, 133.0)
- added R11: R_US, Resistor_SMD:R_0603_1608Metric, F.Cu at (147.0, 141.2)
- added R15: R_US, Resistor_SMD:R_0603_1608Metric, B.Cu at (143.3, 142.1)
- added R5: R_US, Resistor_SMD:R_0603_1608Metric, B.Cu at (139.3, 131.2)
- added R8: R_US, Resistor_SMD:R_0603_1608Metric, F.Cu at (149.0, 141.2)
- added REF**: OSHW-Logo2_7.3x6mm_SilkScreen, Symbol:OSHW-Logo2_7.3x6mm_SilkScreen, B.Cu at (121.8, 90.6)
- added REF**: KiCad-Logo_5mm_SilkScreen, Symbol:KiCad-Logo_5mm_SilkScreen, B.Cu at (146.1, 90.7)
- C13, C9, U4: moved to F.Cu
- J4: value Control -> Conn_01x04_Female; footprint Connector_PinHeader_1.27mm:PinHeader_1x06_P1.27mm_Vertical -> Connector_PinHeader_2.54mm:PinHeader_1x04_P2.54mm_Vertical
- R1, R2, R3: value PSR400ITQFL3L00 -> WSLF25121L000FEB; footprint SamacSys_Parts:RESC10052X200N -> SamacSys_Parts:RESC6430X38N
- R10, R12, R4, R6, R7, R9: value R_US -> 10
- R13: value 10k -> R_US; moved to F.Cu
- R14: value 10k -> R_US
- moved Y1 92.5 mm to (132.5, 134.6), turned to 180 degrees
- moved C13 87.0 mm to (126.7, 143.1), turned to 90 degrees
- moved C9 77.1 mm to (132.2, 143.1), turned to -90 degrees
- moved J4 73.4 mm to (148.3, 145.8)
- moved C11 70.5 mm to (142.2, 134.2), turned to 0 degrees
- moved C12 70.0 mm to (151.4, 131.1), turned to 0 degrees
- moved J8 68.6 mm to (129.9, 143.6)
- moved U4 66.3 mm to (129.5, 142.9), turned to 180 degrees
- moved R14 64.3 mm to (145.8, 142.1), turned to -90 degrees
- moved J7 51.9 mm to (143.0, 138.4), turned to 0 degrees
- moved IC1 42.3 mm to (137.3, 135.3), turned to -90 degrees
- moved C10 32.8 mm to (132.6, 132.8), turned to 180 degrees
- moved R13 22.0 mm to (145.0, 141.2), turned to 90 degrees
- moved R2 12.4 mm to (134.8, 126.6)
- moved R1 12.3 mm to (147.0, 126.5)
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Connections:
- C10 pad 1: /Controller/VDD -> /VDD
- C11 pad 1: /Controller/VDD -> /VDD
- C12 pad 1: /Controller/VDD -> /VDD
- C13 pad 1: /Controller/VDD -> /VDD
- IC1 pad 10: unconnected-(IC1-Pad10) -> /Controller/I_{SENSE}A
- IC1 pad 11: /Controller/VDD -> /VDD
- IC1 pad 12: /Controller/BL -> /Controller/AL
- IC1 pad 13: /Controller/BH -> /Controller/AH
- IC1 pad 14: /Controller/AL -> /Controller/HALL_C
- IC1 pad 15: /Controller/AH -> /Controller/HALL_B
- IC1 pad 16: unconnected-(IC1-Pad16) -> /Controller/HALL_A
- IC1 pad 17: /Controller/VDD -> /VDD
- IC1 pad 18: /Controller/VDD -> /VDD
- IC1 pad 2: /Controller/VDD -> /VDD
- IC1 pad 21: /Controller/CS -> unconnected-(IC1-Pad21)
- IC1 pad 22: /Controller/SCLK -> unconnected-(IC1-Pad22)
- IC1 pad 23: /Controller/MOSI -> /Controller/SCL
- IC1 pad 24: /Controller/MISO -> /Controller/SDA
- IC1 pad 27: unconnected-(IC1-Pad27) -> /Controller/CL
- IC1 pad 28: unconnected-(IC1-Pad28) -> /Controller/CH
- IC1 pad 3: /Controller/VDD -> /VDD
- IC1 pad 31: /Controller/VDD -> /VDD
- IC1 pad 32: /Controller/VDD -> /VDD
- IC1 pad 4: /Controller/HALL_A -> /Controller/BL
- IC1 pad 5: /Controller/HALL_B -> /Controller/BH
- IC1 pad 6: /Controller/HALL_C -> /Controller/RST
- IC1 pad 8: /Controller/I_{SENSE} -> /Controller/I_{SENSE}B
- IC1 pad 9: /Controller/V_{TEMP} -> /Controller/I_{SENSE}C
- IC4 pad 2: /Controller/I_{SENSE} -> /Controller/I_{SENSE}A
- IC4 pad 4: /Driver FETs/IS -> /Driver FETs/ISA
- J4 pad 2: /Controller/CS -> /Controller/SCL
- J4 pad 3: /Controller/SCLK -> /Controller/SDA
- J4 pad 4: /Controller/MISO -> /VDD
- J7 pad 2: /Controller/HALL_C -> /Controller/HALL_A
- J7 pad 4: /Controller/HALL_A -> /Controller/HALL_C
- Q10 pad 1: /Driver FETs/IS -> /Driver FETs/ISC
- Q10 pad 2: /Driver FETs/IS -> /Driver FETs/ISC
- Q10 pad 3: /Driver FETs/IS -> /Driver FETs/ISC
- Q12 pad 1: /Driver FETs/IS -> /Driver FETs/ISC
- Q12 pad 2: /Driver FETs/IS -> /Driver FETs/ISC
- Q12 pad 3: /Driver FETs/IS -> /Driver FETs/ISC
- Q2 pad 1: /Driver FETs/IS -> /Driver FETs/ISA
- Q2 pad 2: /Driver FETs/IS -> /Driver FETs/ISA
- Q2 pad 3: /Driver FETs/IS -> /Driver FETs/ISA
- Q4 pad 1: /Driver FETs/IS -> /Driver FETs/ISA
- Q4 pad 2: /Driver FETs/IS -> /Driver FETs/ISA
- Q4 pad 3: /Driver FETs/IS -> /Driver FETs/ISA
- Q6 pad 1: /Driver FETs/IS -> /Driver FETs/ISB
- Q6 pad 2: /Driver FETs/IS -> /Driver FETs/ISB
- Q6 pad 3: /Driver FETs/IS -> /Driver FETs/ISB
- Q8 pad 1: /Driver FETs/IS -> /Driver FETs/ISB
- Q8 pad 2: /Driver FETs/IS -> /Driver FETs/ISB
- Q8 pad 3: /Driver FETs/IS -> /Driver FETs/ISB
- R1 pad 2: /Driver FETs/IS -> /Driver FETs/ISA
- R13 pad 1: /Controller/3V3USB -> /VDD
- R13 pad 2: Net-(Q13-Pad3) -> /Controller/HALL_A
- R14 pad 1: /Controller/3V3 -> /VDD
- R14 pad 2: Net-(Q15-Pad3) -> /Controller/SCL
- R2 pad 2: /Driver FETs/IS -> /Driver FETs/ISB
- R3 pad 2: /Driver FETs/IS -> /Driver FETs/ISC
- U4 pad 1: /Controller/VDD -> /VDD
Routing:
- net /VDD: track 0.00 -> 159.2 mm, vias 0 -> 1
- net /Controller/I_{SENSE}C: track 0.00 -> 21.9 mm, vias 0 -> 2
- net /Controller/I_{SENSE}A: track 0.00 -> 18.9 mm, vias 0 -> 2
- net /Controller/CL: track 0.00 -> 17.9 mm
- net /Controller/CH: track 0.00 -> 16.6 mm
- net /Controller/SCL: track 0.00 -> 15.8 mm
- net /Controller/AH: track 0.00 -> 15.3 mm
- net /Controller/AL: track 0.00 -> 13.7 mm
- net /Controller/SDA: track 0.00 -> 13.4 mm
- net /Driver FETs/IS: track 11.9 -> 0.00 mm, vias 1 -> 0
- net /Pre-Driver/V_{DRIVE}: track 67.7 -> 56.2 mm, vias 3 -> 4
- net /Driver FETs/ISA: track 0.00 -> 6.39 mm, vias 0 -> 1
- net /Controller/BL: track 0.18 -> 6.50 mm
- net /Driver FETs/ISC: track 0.00 -> 6.20 mm, vias 0 -> 1
- net Net-(Q13-Pad3): track 6.07 -> 0.00 mm
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- added copper zone on F.Cu, net /Driver FETs/ISA
- added copper zone on F.Cu, net /Driver FETs/ISB
- added copper zone on F.Cu, net /Driver FETs/ISC
- removed copper zone on F.Cu, net /Driver FETs/IS
Other:
- outline, holes or cut-outs redrawn
- board text added: "GND"
- board text added: "SCL"
- board text added: "SDA"
- board text added: "VDD"
