File: OpenECU/Hardware/OpenECU.kicad_sch (KiCad schematic)
At the start: 1 part

Commit message: updated mc
Parts:
- removed IC?: ESP32-C3, QFN50P500X500X90-33N-D, symbol SamacSys_Parts:ESP32-C3
Other:
- added sheet MCU (MCU.kicad_sch)
- added sheet Sensors (Sensors.kicad_sch)
- added sheet USB (USB.kicad_sch)
- added sheet Voltage Generation (VGen.kicad_sch)
Changed lines of the file:
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@@
 (kicad_sch (version 20211123) (generator eeschema)
   (paper "A4")
-  (symbol (lib_id "SamacSys_Parts:ESP32-C3") (at 110.49 82.55 0) (unit 1)
-    (in_bom yes) (on_board yes) (fields_autoplaced)
-    (property "Reference" "IC?" (id 0) (at 156.9703 76.5767 0))
-    (property "Value" "ESP32-C3" (id 1) (at 156.9703 79.3518 0))
-    (property "Footprint" "QFN50P500X500X90-33N-D" (id 2) (at 152.4 69.85 0)
-      (effects (font (size 1.27 1.27)) (justify left) hide)
+  (sheet (at 104.14 41.91) (size 38.1 24.13) (fields_autoplaced)
+    (stroke (width 0.1524) (type solid) (color 0 0 0 0))
+    (fill (color 0 0 0 0.0000))
+    (property "Sheet name" "MCU" (id 0) (at 104.14 41.1984 0)
+      (effects (font (size 1.27 1.27)) (justify left bottom))
     )
-    (property "Datasheet" "https://www.espressif.com/sites/default/files/documentation/esp32-c3_datasheet_en.pdf" (id 3) (at 152.4 72.39 0)
-      (effects (font (size 1.27 1.27)) (justify left) hide)
+    (property "Sheet file" "MCU.kicad_sch" (id 1) (at 104.14 66.6246 0)
+      (effects (font (size 1.27 1.27)) (justify left top))
     )
-    (property "Description" "Ultra-Low-Power SoC with RISC-V Single-Core CPU" (id 4) (at 152.4 74.93 0)
-      (effects (font (size 1.27 1.27)) (justify left) hide)
+  )
+  (sheet (at 68.58 41.91) (size 21.59 24.13) (fields_autoplaced)
+    (stroke (width 0.1524) (type solid) (color 0 0 0 0))
+    (fill (color 0 0 0 0.0000))
+    (property "Sheet name" "USB" (id 0) (at 68.58 41.1984 0)
+      (effects (font (size 1.27 1.27)) (justify left bottom))
     )
-    (property "Height" "0.9" (id 5) (at 152.4 77.47 0)
-      (effects (font (size 1.27 1.27)) (justify left) hide)
+    (property "Sheet file" "USB.kicad_sch" (id 1) (at 68.58 66.6246 0)
+      (effects (font (size 1.27 1.27)) (justify left top))
     )
-    (property "Mouser Part Number" "356-ESP32-C3" (id 6) (at 152.4 80.01 0)
-      (effects (font (size 1.27 1.27)) (justify left) hide)
+  )
+  (sheet (at 152.4 41.91) (size 30.48 24.13) (fields_autoplaced)
+    (stroke (width 0.1524) (type solid) (color 0 0 0 0))
+    (fill (color 0 0 0 0.0000))
+    (property "Sheet name" "Sensors" (id 0) (at 152.4 41.1984 0)
+      (effects (font (size 1.27 1.27)) (justify left bottom))
     )
-    (property "Mouser Price/Stock" "https://www.mouser.co.uk/ProductDetail/Espressif-Systems/ESP32-C3?qs=iLbezkQI%252BsiMXe7tMG%252Bo%2FA%3D%3D" (id 7) (at 152.4 82.55 0)
-      (effects (font (size 1.27 1.27)) (justify left) hide)
+    (property "Sheet file" "Sensors.kicad_sch" (id 1) (at 152.4 66.6246 0)
+      (effects (font (size 1.27 1.27)) (justify left top))
     )
-    (property "Manufacturer_Name" "Espressif Systems" (id 8) (at 152.4 85.09 0)
-      (effects (font (size 1.27 1.27)) (justify left) hide)
+  )
+  (sheet (at 68.58 74.93) (size 21.59 24.13) (fields_autoplaced)
+    (stroke (width 0.1524) (type solid) (color 0 0 0 0))
+    (fill (color 0 0 0 0.0000))
+    (property "Sheet name" "Voltage Generation" (id 0) (at 68.58 74.2184 0)
+      (effects (font (size 1.27 1.27)) (justify left bottom))
     )
-    (property "Manufacturer_Part_Number" "ESP32-C3" (id 9) (at 152.4 87.63 0)
-      (effects (font (size 1.27 1.27)) (justify left) hide)
+    (property "Sheet file" "VGen.kicad_sch" (id 1) (at 68.58 99.6446 0)
+      (effects (font (size 1.27 1.27)) (justify left top))
     )
-    (pin "1")
-    (pin "10")
-    (pin "11")
-    (pin "12")
-    (pin "13")
-    (pin "14")
-    (pin "15")
-    (pin "16")
-    (pin "17")
-    (pin "18")
-    (pin "19")
-    (pin "2")
-    (pin "20")
-    (pin "21")
-    (pin "22")
-    (pin "23")
-    (pin "24")
-    (pin "25")
-    (pin "26")
-    (pin "27")
-    (pin "28")
-    (pin "29")
-    (pin "3")
-    (pin "30")
-    (pin "31")
-    (pin "32")
-    (pin "33")
-    (pin "4")
-    (pin "5")
-    (pin "6")
-    (pin "7")
-    (pin "8")
-    (pin "9")
   )
   (sheet_instances
     (path "/" (page "1"))
+    (path "/a22ef832-33fc-4544-9dac-b6ed3c7ca675" (page "2"))
+    (path "/381ac0ba-1452-42d2-80b0-a1b73edf92b7" (page "3"))
+    (path "/7ba41709-763d-4924-b365-501a763cce07" (page "4"))
+    (path "/a54d34e1-6045-4f4c-bb09-a70ef04dc72a" (page "5"))
   )
   (symbol_instances
-    (path "/14c24f6d-c2bf-4b01-9d4b-7f0755e08445"
-      (reference "IC?") (unit 1) (value "ESP32-C3") (footprint "QFN50P500X500X90-33N-D")
+    (path "/381ac0ba-1452-42d2-80b0-a1b73edf92b7/1112b7d9-fa55-49d2-a6fe-e666f391852c"
+      (reference "U?") (unit 1) (value "ESP32-C3-WROOM-02-H4") (footprint "MODULE_ESP32-C3-WROOM-02-H4")
     )
   )
