File: OpenMC/Hardware/Controller.kicad_sch (KiCad schematic)
At the start: 15 parts, among them IC1 ESP32-C3, J8 216990-0001, U4 LM3480-3.3, Y1 40MHz

Commit message: updated footprint
Parts:
- IC1: footprint QFN50P500X500X90-33N-D -> Package_DFN_QFN:QFN-32-1EP_5x5mm_P0.5mm_EP3.7x3.7mm
Changed lines of the file:
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@@
     (property "Reference" "IC1" (id 0) (at 101.0903 112.1367 0))
     (property "Value" "ESP32-C3" (id 1) (at 101.0903 114.9118 0))
-    (property "Footprint" "QFN50P500X500X90-33N-D" (id 2) (at 96.52 105.41 0)
+    (property "Footprint" "Package_DFN_QFN:QFN-32-1EP_5x5mm_P0.5mm_EP3.7x3.7mm" (id 2) (at 96.52 105.41 0)
       (effects (font (size 1.27 1.27)) (justify left) hide)
     )
