File: OpenMC/Hardware/Hi-LowDriver.kicad_sch (KiCad schematic)
At the start: 6 parts, among them U1 LT2190NTR

Commit message: updated footprint
Parts:
- renumbered C5 to C15, C1 to C3, D1 to D3, R4 to R10, R6 to R12, U1 to U3
Changed lines of the file:
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@@
   (symbol (lib_id "OpenMC:LT2190NTR") (at 149.86 99.06 0)
     (in_bom yes) (on_board yes) (fields_autoplaced)
-    (property "Reference" "U1" (id 0) (at 149.86 88.7943 0))
+    (property "Reference" "U3" (id 0) (at 149.86 88.7943 0))
     (property "Value" "LT2190NTR" (id 1) (at 149.86 91.5694 0))
     (property "Footprint" "Package_SO:SOIC-8_3.9x4.9mm_P1.27mm" (id 2) (at 147.32 99.06 0)
@@
   (symbol (lib_id "Device:C_Small") (at 161.29 105.41 0)
     (in_bom yes) (on_board yes)
-    (property "Reference" "C5" (id 0) (at 163.6141 104.5078 0)
+    (property "Reference" "C15" (id 0) (at 163.6141 104.5078 0)
       (effects (font (size 1.27 1.27)) (justify left))
     )
@@
   (symbol (lib_id "Device:R_US") (at 137.16 102.87 90)
     (in_bom yes) (on_board yes)
-    (property "Reference" "R4" (id 0) (at 137.16 105.41 90))
+    (property "Reference" "R10" (id 0) (at 137.16 105.41 90))
     (property "Value" "10" (id 1) (at 137.16 100.7896 90)
       (effects (font (size 1.27 1.27)) hide)
@@
   (symbol (lib_id "Device:C_Small") (at 173.99 97.79 0)
     (in_bom yes) (on_board yes)
-    (property "Reference" "C1" (id 0) (at 176.3141 96.8878 0)
+    (property "Reference" "C3" (id 0) (at 176.3141 96.8878 0)
       (effects (font (size 1.27 1.27)) (justify left))
     )
@@
   (symbol (lib_id "Device:D") (at 161.29 91.44 90)
     (in_bom yes) (on_board yes) (fields_autoplaced)
-    (property "Reference" "D1" (id 0) (at 163.322 90.5315 90)
+    (property "Reference" "D3" (id 0) (at 163.322 90.5315 90)
       (effects (font (size 1.27 1.27)) (justify right))
     )
@@
   (symbol (lib_id "Device:R_US") (at 162.56 97.79 90)
     (in_bom yes) (on_board yes)
-    (property "Reference" "R6" (id 0) (at 165.1 96.52 90))
+    (property "Reference" "R12" (id 0) (at 165.1 96.52 90))
     (property "Value" "10" (id 1) (at 162.56 95.7096 90)
       (effects (font (size 1.27 1.27)) hide)
